File: cm2.kicad_pcb (KiCad board)
At the start: 2 copper layers, 16 parts

Commit message: checkpoint
Parts:
- removed D00@1, D01@1, D02@1, D03@1: LED_Small_ALT, LED_THT:LED_D5.0mm
- added D00D1: LED_Small_ALT, LED_THT:LED_D5.0mm, F.Cu at (0.00, 47.6)
- added D01D1: LED_Small_ALT, LED_THT:LED_D5.0mm, F.Cu at (15.9, 47.6)
- added D02D1: LED_Small_ALT, LED_THT:LED_D5.0mm, F.Cu at (31.8, 47.6)
- added D03D1: LED_Small_ALT, LED_THT:LED_D5.0mm, F.Cu at (47.6, 47.6)
- moved D00A1 15.9 mm to (0.00, 0.00)
- moved D00B1 15.9 mm to (0.00, 15.9)
- moved D00C1 15.9 mm to (0.00, 31.8)
- moved D01A1 15.9 mm to (15.9, 0.00)
- moved D01B1 15.9 mm to (15.9, 15.9)
- moved D01C1 15.9 mm to (15.9, 31.8)
- moved D02A1 15.9 mm to (31.8, 0.00)
- moved D02B1 15.9 mm to (31.8, 15.9)
- moved D02C1 15.9 mm to (31.8, 31.8)
- moved D03A1 15.9 mm to (47.6, 0.00)
- moved D03B1 15.9 mm to (47.6, 15.9)
- moved D03C1 15.9 mm to (47.6, 31.8)
Connections:
- D00A1 pad 1: /col02 -> /col00
- D00A1 pad 2: /row1 -> /row0
- D00B1 pad 1: /col03 -> /col01
- D00B1 pad 2: /row1 -> /row0
- D00C1 pad 1: /col04 -> /col02
- D00C1 pad 2: /row1 -> /row0
- D01A1 pad 1: /col02 -> /col00
- D01A1 pad 2: /row2 -> /row1
- D01B1 pad 1: /col03 -> /col01
- D01B1 pad 2: /row2 -> /row1
- D01C1 pad 1: /col04 -> /col02
- D01C1 pad 2: /row2 -> /row1
- D02A1 pad 1: /col02 -> /col00
- D02A1 pad 2: /row3 -> /row2
- D02B1 pad 1: /col03 -> /col01
- D02B1 pad 2: /row3 -> /row2
- D02C1 pad 1: /col04 -> /col02
- D02C1 pad 2: /row3 -> /row2
- D03A1 pad 1: /col02 -> /col00
- D03A1 pad 2: /row4 -> /row3
- D03B1 pad 1: /col03 -> /col01
- D03B1 pad 2: /row4 -> /row3
- D03C1 pad 1: /col04 -> /col02
- D03C1 pad 2: /row4 -> /row3

Commit message: checkpoint
Parts:
- added D00A2: LED_Small_ALT, LED_THT:LED_D5.0mm, F.Cu at (0.00, 127.0)
- added D00B2: LED_Small_ALT, LED_THT:LED_D5.0mm, F.Cu at (0.00, 142.9)
- added D00C2: LED_Small_ALT, LED_THT:LED_D5.0mm, F.Cu at (0.00, 158.8)
- added D00D2: LED_Small_ALT, LED_THT:LED_D5.0mm, F.Cu at (0.00, 174.6)
- added D00E1: LED_Small_ALT, LED_THT:LED_D5.0mm, F.Cu at (0.00, 63.5)
- added D00E2: LED_Small_ALT, LED_THT:LED_D5.0mm, F.Cu at (0.00, 190.5)
- added D00F1: LED_Small_ALT, LED_THT:LED_D5.0mm, F.Cu at (0.00, 79.4)
- added D00F2: LED_Small_ALT, LED_THT:LED_D5.0mm, F.Cu at (0.00, 206.4)
- added D00G1: LED_Small_ALT, LED_THT:LED_D5.0mm, F.Cu at (0.00, 95.2)
- added D00G2: LED_Small_ALT, LED_THT:LED_D5.0mm, F.Cu at (0.00, 222.2)
- added D00H1: LED_Small_ALT, LED_THT:LED_D5.0mm, F.Cu at (0.00, 111.1)
- added D00H2: LED_Small_ALT, LED_THT:LED_D5.0mm, F.Cu at (0.00, 238.1)
- added D01A2: LED_Small_ALT, LED_THT:LED_D5.0mm, F.Cu at (15.9, 127.0)
- added D01B2: LED_Small_ALT, LED_THT:LED_D5.0mm, F.Cu at (15.9, 142.9)
- added D01C2: LED_Small_ALT, LED_THT:LED_D5.0mm, F.Cu at (15.9, 158.8)
- added D01D2: LED_Small_ALT, LED_THT:LED_D5.0mm, F.Cu at (15.9, 174.6)
- added D01E1: LED_Small_ALT, LED_THT:LED_D5.0mm, F.Cu at (15.9, 63.5)
- added D01E2: LED_Small_ALT, LED_THT:LED_D5.0mm, F.Cu at (15.9, 190.5)
- added D01F1: LED_Small_ALT, LED_THT:LED_D5.0mm, F.Cu at (15.9, 79.4)
- added D01F2: LED_Small_ALT, LED_THT:LED_D5.0mm, F.Cu at (15.9, 206.4)
- added D01G1: LED_Small_ALT, LED_THT:LED_D5.0mm, F.Cu at (15.9, 95.2)
- added D01G2: LED_Small_ALT, LED_THT:LED_D5.0mm, F.Cu at (15.9, 222.2)
- added D01H1: LED_Small_ALT, LED_THT:LED_D5.0mm, F.Cu at (15.9, 111.1)
- added D01H2: LED_Small_ALT, LED_THT:LED_D5.0mm, F.Cu at (15.9, 238.1)
- added D02A2: LED_Small_ALT, LED_THT:LED_D5.0mm, F.Cu at (31.8, 127.0)
- added D02B2: LED_Small_ALT, LED_THT:LED_D5.0mm, F.Cu at (31.8, 142.9)
- added D02C2: LED_Small_ALT, LED_THT:LED_D5.0mm, F.Cu at (31.8, 158.8)
- added D02D2: LED_Small_ALT, LED_THT:LED_D5.0mm, F.Cu at (31.8, 174.6)
- added D02E1: LED_Small_ALT, LED_THT:LED_D5.0mm, F.Cu at (31.8, 63.5)
- added D02E2: LED_Small_ALT, LED_THT:LED_D5.0mm, F.Cu at (31.8, 190.5)
- added D02F1: LED_Small_ALT, LED_THT:LED_D5.0mm, F.Cu at (31.8, 79.4)
- added D02F2: LED_Small_ALT, LED_THT:LED_D5.0mm, F.Cu at (31.8, 206.4)
- added D02G1: LED_Small_ALT, LED_THT:LED_D5.0mm, F.Cu at (31.8, 95.2)
- added D02G2: LED_Small_ALT, LED_THT:LED_D5.0mm, F.Cu at (31.8, 222.2)
- added D02H1: LED_Small_ALT, LED_THT:LED_D5.0mm, F.Cu at (31.8, 111.1)
- added D02H2: LED_Small_ALT, LED_THT:LED_D5.0mm, F.Cu at (31.8, 238.1)
- added D03A2: LED_Small_ALT, LED_THT:LED_D5.0mm, F.Cu at (47.6, 127.0)
- added D03B2: LED_Small_ALT, LED_THT:LED_D5.0mm, F.Cu at (47.6, 142.9)
- added D03C2: LED_Small_ALT, LED_THT:LED_D5.0mm, F.Cu at (47.6, 158.8)
- added D03D2: LED_Small_ALT, LED_THT:LED_D5.0mm, F.Cu at (47.6, 174.6)
- added D03E1: LED_Small_ALT, LED_THT:LED_D5.0mm, F.Cu at (47.6, 63.5)
- added D03E2: LED_Small_ALT, LED_THT:LED_D5.0mm, F.Cu at (47.6, 190.5)
- added D03F1: LED_Small_ALT, LED_THT:LED_D5.0mm, F.Cu at (47.6, 79.4)
- added D03F2: LED_Small_ALT, LED_THT:LED_D5.0mm, F.Cu at (47.6, 206.4)
- added D03G1: LED_Small_ALT, LED_THT:LED_D5.0mm, F.Cu at (47.6, 95.2)
- added D03G2: LED_Small_ALT, LED_THT:LED_D5.0mm, F.Cu at (47.6, 222.2)
- added D03H1: LED_Small_ALT, LED_THT:LED_D5.0mm, F.Cu at (47.6, 111.1)
- added D03H2: LED_Small_ALT, LED_THT:LED_D5.0mm, F.Cu at (47.6, 238.1)
- added D04A1: LED_Small_ALT, LED_THT:LED_D5.0mm, F.Cu at (63.5, 0.00)
- added D04A2: LED_Small_ALT, LED_THT:LED_D5.0mm, F.Cu at (63.5, 127.0)
- added D04B1: LED_Small_ALT, LED_THT:LED_D5.0mm, F.Cu at (63.5, 15.9)
- added D04B2: LED_Small_ALT, LED_THT:LED_D5.0mm, F.Cu at (63.5, 142.9)
- added D04C1: LED_Small_ALT, LED_THT:LED_D5.0mm, F.Cu at (63.5, 31.8)
- added D04C2: LED_Small_ALT, LED_THT:LED_D5.0mm, F.Cu at (63.5, 158.8)
- added D04D1: LED_Small_ALT, LED_THT:LED_D5.0mm, F.Cu at (63.5, 47.6)
- added D04D2: LED_Small_ALT, LED_THT:LED_D5.0mm, F.Cu at (63.5, 174.6)
- added D04E1: LED_Small_ALT, LED_THT:LED_D5.0mm, F.Cu at (63.5, 63.5)
- added D04E2: LED_Small_ALT, LED_THT:LED_D5.0mm, F.Cu at (63.5, 190.5)
- added D04F1: LED_Small_ALT, LED_THT:LED_D5.0mm, F.Cu at (63.5, 79.4)
- added D04F2: LED_Small_ALT, LED_THT:LED_D5.0mm, F.Cu at (63.5, 206.4)
- added D04G1: LED_Small_ALT, LED_THT:LED_D5.0mm, F.Cu at (63.5, 95.2)
- added D04G2: LED_Small_ALT, LED_THT:LED_D5.0mm, F.Cu at (63.5, 222.2)
- added D04H1: LED_Small_ALT, LED_THT:LED_D5.0mm, F.Cu at (63.5, 111.1)
- added D04H2: LED_Small_ALT, LED_THT:LED_D5.0mm, F.Cu at (63.5, 238.1)
- added D05A1: LED_Small_ALT, LED_THT:LED_D5.0mm, F.Cu at (79.4, 0.00)
- added D05A2: LED_Small_ALT, LED_THT:LED_D5.0mm, F.Cu at (79.4, 127.0)
- added D05B1: LED_Small_ALT, LED_THT:LED_D5.0mm, F.Cu at (79.4, 15.9)
- added D05B2: LED_Small_ALT, LED_THT:LED_D5.0mm, F.Cu at (79.4, 142.9)
- added D05C1: LED_Small_ALT, LED_THT:LED_D5.0mm, F.Cu at (79.4, 31.8)
- added D05C2: LED_Small_ALT, LED_THT:LED_D5.0mm, F.Cu at (79.4, 158.8)
- added D05D1: LED_Small_ALT, LED_THT:LED_D5.0mm, F.Cu at (79.4, 47.6)
- added D05D2: LED_Small_ALT, LED_THT:LED_D5.0mm, F.Cu at (79.4, 174.6)
- added D05E1: LED_Small_ALT, LED_THT:LED_D5.0mm, F.Cu at (79.4, 63.5)
- added D05E2: LED_Small_ALT, LED_THT:LED_D5.0mm, F.Cu at (79.4, 190.5)
- added D05F1: LED_Small_ALT, LED_THT:LED_D5.0mm, F.Cu at (79.4, 79.4)
- added D05F2: LED_Small_ALT, LED_THT:LED_D5.0mm, F.Cu at (79.4, 206.4)
- added D05G1: LED_Small_ALT, LED_THT:LED_D5.0mm, F.Cu at (79.4, 95.2)
- added D05G2: LED_Small_ALT, LED_THT:LED_D5.0mm, F.Cu at (79.4, 222.2)
- added D05H1: LED_Small_ALT, LED_THT:LED_D5.0mm, F.Cu at (79.4, 111.1)
- added D05H2: LED_Small_ALT, LED_THT:LED_D5.0mm, F.Cu at (79.4, 238.1)
- added D06A1: LED_Small_ALT, LED_THT:LED_D5.0mm, F.Cu at (95.2, 0.00)
- added D06A2: LED_Small_ALT, LED_THT:LED_D5.0mm, F.Cu at (95.2, 127.0)
- added D06B1: LED_Small_ALT, LED_THT:LED_D5.0mm, F.Cu at (95.2, 15.9)
- added D06B2: LED_Small_ALT, LED_THT:LED_D5.0mm, F.Cu at (95.2, 142.9)
- added D06C1: LED_Small_ALT, LED_THT:LED_D5.0mm, F.Cu at (95.2, 31.8)
- added D06C2: LED_Small_ALT, LED_THT:LED_D5.0mm, F.Cu at (95.2, 158.8)
- added D06D1: LED_Small_ALT, LED_THT:LED_D5.0mm, F.Cu at (95.2, 47.6)
- added D06D2: LED_Small_ALT, LED_THT:LED_D5.0mm, F.Cu at (95.2, 174.6)
- added D06E1: LED_Small_ALT, LED_THT:LED_D5.0mm, F.Cu at (95.2, 63.5)
- added D06E2: LED_Small_ALT, LED_THT:LED_D5.0mm, F.Cu at (95.2, 190.5)
- added D06F1: LED_Small_ALT, LED_THT:LED_D5.0mm, F.Cu at (95.2, 79.4)
- added D06F2: LED_Small_ALT, LED_THT:LED_D5.0mm, F.Cu at (95.2, 206.4)
- added D06G1: LED_Small_ALT, LED_THT:LED_D5.0mm, F.Cu at (95.2, 95.2)
- added D06G2: LED_Small_ALT, LED_THT:LED_D5.0mm, F.Cu at (95.2, 222.2)
- added D06H1: LED_Small_ALT, LED_THT:LED_D5.0mm, F.Cu at (95.2, 111.1)
- added D06H2: LED_Small_ALT, LED_THT:LED_D5.0mm, F.Cu at (95.2, 238.1)
- added D07A1: LED_Small_ALT, LED_THT:LED_D5.0mm, F.Cu at (111.1, 0.00)
- added D07A2: LED_Small_ALT, LED_THT:LED_D5.0mm, F.Cu at (111.1, 127.0)
- added D07B1: LED_Small_ALT, LED_THT:LED_D5.0mm, F.Cu at (111.1, 15.9)
- added D07B2: LED_Small_ALT, LED_THT:LED_D5.0mm, F.Cu at (111.1, 142.9)
- added D07C1: LED_Small_ALT, LED_THT:LED_D5.0mm, F.Cu at (111.1, 31.8)
- added D07C2: LED_Small_ALT, LED_THT:LED_D5.0mm, F.Cu at (111.1, 158.8)
- added D07D1: LED_Small_ALT, LED_THT:LED_D5.0mm, F.Cu at (111.1, 47.6)
- added D07D2: LED_Small_ALT, LED_THT:LED_D5.0mm, F.Cu at (111.1, 174.6)
- added D07E1: LED_Small_ALT, LED_THT:LED_D5.0mm, F.Cu at (111.1, 63.5)
- added D07E2: LED_Small_ALT, LED_THT:LED_D5.0mm, F.Cu at (111.1, 190.5)
- added D07F1: LED_Small_ALT, LED_THT:LED_D5.0mm, F.Cu at (111.1, 79.4)
- added D07F2: LED_Small_ALT, LED_THT:LED_D5.0mm, F.Cu at (111.1, 206.4)
- added D07G1: LED_Small_ALT, LED_THT:LED_D5.0mm, F.Cu at (111.1, 95.2)
- added D07G2: LED_Small_ALT, LED_THT:LED_D5.0mm, F.Cu at (111.1, 222.2)
- added D07H1: LED_Small_ALT, LED_THT:LED_D5.0mm, F.Cu at (111.1, 111.1)
- added D07H2: LED_Small_ALT, LED_THT:LED_D5.0mm, F.Cu at (111.1, 238.1)
- added D08A1: LED_Small_ALT, LED_THT:LED_D5.0mm, F.Cu at (127.0, 0.00)
- added D08A2: LED_Small_ALT, LED_THT:LED_D5.0mm, F.Cu at (127.0, 127.0)
- added D08B1: LED_Small_ALT, LED_THT:LED_D5.0mm, F.Cu at (127.0, 15.9)
- added D08B2: LED_Small_ALT, LED_THT:LED_D5.0mm, F.Cu at (127.0, 142.9)
- added D08C1: LED_Small_ALT, LED_THT:LED_D5.0mm, F.Cu at (127.0, 31.8)
- added D08C2: LED_Small_ALT, LED_THT:LED_D5.0mm, F.Cu at (127.0, 158.8)
- added D08D1: LED_Small_ALT, LED_THT:LED_D5.0mm, F.Cu at (127.0, 47.6)
- added D08D2: LED_Small_ALT, LED_THT:LED_D5.0mm, F.Cu at (127.0, 174.6)
- added D08E1: LED_Small_ALT, LED_THT:LED_D5.0mm, F.Cu at (127.0, 63.5)
- added D08E2: LED_Small_ALT, LED_THT:LED_D5.0mm, F.Cu at (127.0, 190.5)
- added D08F1: LED_Small_ALT, LED_THT:LED_D5.0mm, F.Cu at (127.0, 79.4)
- added D08F2: LED_Small_ALT, LED_THT:LED_D5.0mm, F.Cu at (127.0, 206.4)
- added D08G1: LED_Small_ALT, LED_THT:LED_D5.0mm, F.Cu at (127.0, 95.2)
- added D08G2: LED_Small_ALT, LED_THT:LED_D5.0mm, F.Cu at (127.0, 222.2)
- added D08H1: LED_Small_ALT, LED_THT:LED_D5.0mm, F.Cu at (127.0, 111.1)
- added D08H2: LED_Small_ALT, LED_THT:LED_D5.0mm, F.Cu at (127.0, 238.1)
- added D09A1: LED_Small_ALT, LED_THT:LED_D5.0mm, F.Cu at (142.9, 0.00)
- added D09A2: LED_Small_ALT, LED_THT:LED_D5.0mm, F.Cu at (142.9, 127.0)
- added D09B1: LED_Small_ALT, LED_THT:LED_D5.0mm, F.Cu at (142.9, 15.9)
- added D09B2: LED_Small_ALT, LED_THT:LED_D5.0mm, F.Cu at (142.9, 142.9)
- added D09C1: LED_Small_ALT, LED_THT:LED_D5.0mm, F.Cu at (142.9, 31.8)
- added D09C2: LED_Small_ALT, LED_THT:LED_D5.0mm, F.Cu at (142.9, 158.8)
- added D09D1: LED_Small_ALT, LED_THT:LED_D5.0mm, F.Cu at (142.9, 47.6)
- added D09D2: LED_Small_ALT, LED_THT:LED_D5.0mm, F.Cu at (142.9, 174.6)
- added D09E1: LED_Small_ALT, LED_THT:LED_D5.0mm, F.Cu at (142.9, 63.5)
- added D09E2: LED_Small_ALT, LED_THT:LED_D5.0mm, F.Cu at (142.9, 190.5)
- added D09F1: LED_Small_ALT, LED_THT:LED_D5.0mm, F.Cu at (142.9, 79.4)
- added D09F2: LED_Small_ALT, LED_THT:LED_D5.0mm, F.Cu at (142.9, 206.4)
- added D09G1: LED_Small_ALT, LED_THT:LED_D5.0mm, F.Cu at (142.9, 95.2)
- added D09G2: LED_Small_ALT, LED_THT:LED_D5.0mm, F.Cu at (142.9, 222.2)
- added D09H1: LED_Small_ALT, LED_THT:LED_D5.0mm, F.Cu at (142.9, 111.1)
- added D09H2: LED_Small_ALT, LED_THT:LED_D5.0mm, F.Cu at (142.9, 238.1)
- added D10A1: LED_Small_ALT, LED_THT:LED_D5.0mm, F.Cu at (158.8, 0.00)
- added D10A2: LED_Small_ALT, LED_THT:LED_D5.0mm, F.Cu at (158.8, 127.0)
- added D10B1: LED_Small_ALT, LED_THT:LED_D5.0mm, F.Cu at (158.8, 15.9)
- added D10B2: LED_Small_ALT, LED_THT:LED_D5.0mm, F.Cu at (158.8, 142.9)
- added D10C1: LED_Small_ALT, LED_THT:LED_D5.0mm, F.Cu at (158.8, 31.8)
- added D10C2: LED_Small_ALT, LED_THT:LED_D5.0mm, F.Cu at (158.8, 158.8)
- added D10D1: LED_Small_ALT, LED_THT:LED_D5.0mm, F.Cu at (158.8, 47.6)
- added D10D2: LED_Small_ALT, LED_THT:LED_D5.0mm, F.Cu at (158.8, 174.6)
- added D10E1: LED_Small_ALT, LED_THT:LED_D5.0mm, F.Cu at (158.8, 63.5)
- added D10E2: LED_Small_ALT, LED_THT:LED_D5.0mm, F.Cu at (158.8, 190.5)
- added D10F1: LED_Small_ALT, LED_THT:LED_D5.0mm, F.Cu at (158.8, 79.4)
- added D10F2: LED_Small_ALT, LED_THT:LED_D5.0mm, F.Cu at (158.8, 206.4)
- added D10G1: LED_Small_ALT, LED_THT:LED_D5.0mm, F.Cu at (158.8, 95.2)
- added D10G2: LED_Small_ALT, LED_THT:LED_D5.0mm, F.Cu at (158.8, 222.2)
- added D10H1: LED_Small_ALT, LED_THT:LED_D5.0mm, F.Cu at (158.8, 111.1)
- added D10H2: LED_Small_ALT, LED_THT:LED_D5.0mm, F.Cu at (158.8, 238.1)
- added D11A1: LED_Small_ALT, LED_THT:LED_D5.0mm, F.Cu at (174.6, 0.00)
- added D11A2: LED_Small_ALT, LED_THT:LED_D5.0mm, F.Cu at (174.6, 127.0)
- added D11B1: LED_Small_ALT, LED_THT:LED_D5.0mm, F.Cu at (174.6, 15.9)
- added D11B2: LED_Small_ALT, LED_THT:LED_D5.0mm, F.Cu at (174.6, 142.9)
- added D11C1: LED_Small_ALT, LED_THT:LED_D5.0mm, F.Cu at (174.6, 31.8)
- added D11C2: LED_Small_ALT, LED_THT:LED_D5.0mm, F.Cu at (174.6, 158.8)
- added D11D1: LED_Small_ALT, LED_THT:LED_D5.0mm, F.Cu at (174.6, 47.6)
- added D11D2: LED_Small_ALT, LED_THT:LED_D5.0mm, F.Cu at (174.6, 174.6)
- added D11E1: LED_Small_ALT, LED_THT:LED_D5.0mm, F.Cu at (174.6, 63.5)
- added D11E2: LED_Small_ALT, LED_THT:LED_D5.0mm, F.Cu at (174.6, 190.5)
- added D11F1: LED_Small_ALT, LED_THT:LED_D5.0mm, F.Cu at (174.6, 79.4)
- added D11F2: LED_Small_ALT, LED_THT:LED_D5.0mm, F.Cu at (174.6, 206.4)
- added D11G1: LED_Small_ALT, LED_THT:LED_D5.0mm, F.Cu at (174.6, 95.2)
- added D11G2: LED_Small_ALT, LED_THT:LED_D5.0mm, F.Cu at (174.6, 222.2)
- added D11H1: LED_Small_ALT, LED_THT:LED_D5.0mm, F.Cu at (174.6, 111.1)
- added D11H2: LED_Small_ALT, LED_THT:LED_D5.0mm, F.Cu at (174.6, 238.1)
- added D12A1: LED_Small_ALT, LED_THT:LED_D5.0mm, F.Cu at (190.5, 0.00)
- added D12A2: LED_Small_ALT, LED_THT:LED_D5.0mm, F.Cu at (190.5, 127.0)
- added D12B1: LED_Small_ALT, LED_THT:LED_D5.0mm, F.Cu at (190.5, 15.9)
- added D12B2: LED_Small_ALT, LED_THT:LED_D5.0mm, F.Cu at (190.5, 142.9)
- added D12C1: LED_Small_ALT, LED_THT:LED_D5.0mm, F.Cu at (190.5, 31.8)
- added D12C2: LED_Small_ALT, LED_THT:LED_D5.0mm, F.Cu at (190.5, 158.8)
- added D12D1: LED_Small_ALT, LED_THT:LED_D5.0mm, F.Cu at (190.5, 47.6)
- added D12D2: LED_Small_ALT, LED_THT:LED_D5.0mm, F.Cu at (190.5, 174.6)
- added D12E1: LED_Small_ALT, LED_THT:LED_D5.0mm, F.Cu at (190.5, 63.5)
- added D12E2: LED_Small_ALT, LED_THT:LED_D5.0mm, F.Cu at (190.5, 190.5)
- added D12F1: LED_Small_ALT, LED_THT:LED_D5.0mm, F.Cu at (190.5, 79.4)
- added D12F2: LED_Small_ALT, LED_THT:LED_D5.0mm, F.Cu at (190.5, 206.4)
- added D12G1: LED_Small_ALT, LED_THT:LED_D5.0mm, F.Cu at (190.5, 95.2)
- added D12G2: LED_Small_ALT, LED_THT:LED_D5.0mm, F.Cu at (190.5, 222.2)
- added D12H1: LED_Small_ALT, LED_THT:LED_D5.0mm, F.Cu at (190.5, 111.1)
- added D12H2: LED_Small_ALT, LED_THT:LED_D5.0mm, F.Cu at (190.5, 238.1)
- added D13A1: LED_Small_ALT, LED_THT:LED_D5.0mm, F.Cu at (206.4, 0.00)
- added D13A2: LED_Small_ALT, LED_THT:LED_D5.0mm, F.Cu at (206.4, 127.0)
- added D13B1: LED_Small_ALT, LED_THT:LED_D5.0mm, F.Cu at (206.4, 15.9)
- added D13B2: LED_Small_ALT, LED_THT:LED_D5.0mm, F.Cu at (206.4, 142.9)
- added D13C1: LED_Small_ALT, LED_THT:LED_D5.0mm, F.Cu at (206.4, 31.8)
- added D13C2: LED_Small_ALT, LED_THT:LED_D5.0mm, F.Cu at (206.4, 158.8)
- added D13D1: LED_Small_ALT, LED_THT:LED_D5.0mm, F.Cu at (206.4, 47.6)
- added D13D2: LED_Small_ALT, LED_THT:LED_D5.0mm, F.Cu at (206.4, 174.6)
- added D13E1: LED_Small_ALT, LED_THT:LED_D5.0mm, F.Cu at (206.4, 63.5)
- added D13E2: LED_Small_ALT, LED_THT:LED_D5.0mm, F.Cu at (206.4, 190.5)
- added D13F1: LED_Small_ALT, LED_THT:LED_D5.0mm, F.Cu at (206.4, 79.4)
- added D13F2: LED_Small_ALT, LED_THT:LED_D5.0mm, F.Cu at (206.4, 206.4)
- added D13G1: LED_Small_ALT, LED_THT:LED_D5.0mm, F.Cu at (206.4, 95.2)
- added D13G2: LED_Small_ALT, LED_THT:LED_D5.0mm, F.Cu at (206.4, 222.2)
- added D13H1: LED_Small_ALT, LED_THT:LED_D5.0mm, F.Cu at (206.4, 111.1)
- added D13H2: LED_Small_ALT, LED_THT:LED_D5.0mm, F.Cu at (206.4, 238.1)
- added D14A1: LED_Small_ALT, LED_THT:LED_D5.0mm, F.Cu at (222.2, 0.00)
- added D14A2: LED_Small_ALT, LED_THT:LED_D5.0mm, F.Cu at (222.2, 127.0)
- added D14B1: LED_Small_ALT, LED_THT:LED_D5.0mm, F.Cu at (222.2, 15.9)
- added D14B2: LED_Small_ALT, LED_THT:LED_D5.0mm, F.Cu at (222.2, 142.9)
- added D14C1: LED_Small_ALT, LED_THT:LED_D5.0mm, F.Cu at (222.2, 31.8)
- added D14C2: LED_Small_ALT, LED_THT:LED_D5.0mm, F.Cu at (222.2, 158.8)
- added D14D1: LED_Small_ALT, LED_THT:LED_D5.0mm, F.Cu at (222.2, 47.6)
- added D14D2: LED_Small_ALT, LED_THT:LED_D5.0mm, F.Cu at (222.2, 174.6)
- added D14E1: LED_Small_ALT, LED_THT:LED_D5.0mm, F.Cu at (222.2, 63.5)
- added D14E2: LED_Small_ALT, LED_THT:LED_D5.0mm, F.Cu at (222.2, 190.5)
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
Commit message: checkpoint
Parts:
- added J1: Conn_02x06_Counter_Clockwise, Connector_PinHeader_2.54mm:PinHeader_2x06_P2.54mm_Horizontal, F.Cu at (513.1, -1.52)
- added J2: Conn_02x06_Counter_Clockwise, Connector_PinSocket_2.54mm:PinSocket_2x06_P2.54mm_Horizontal, F.Cu at (505.5, 246.1)

Commit message: checkpoint
Parts:
- added J3: Raspberry_Pi_2_3, Connector_PinSocket_2.54mm:PinSocket_2x20_P2.54mm_Vertical, F.Cu at (531.2, 89.3)
Changed lines of the file:
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@@
     (tracks 0)
     (zones 0)
-    (modules 516)
+    (modules 517)
     (nets 83)
   )
@@
     (add_net "Net-(J2-Pad8)")
     (add_net "Net-(J2-Pad9)")
+    (add_net "Net-(J3-Pad1)")
+    (add_net "Net-(J3-Pad10)")
+    (add_net "Net-(J3-Pad11)")
+    (add_net "Net-(J3-Pad12)")
+    (add_net "Net-(J3-Pad13)")
+    (add_net "Net-(J3-Pad14)")
+    (add_net "Net-(J3-Pad15)")
+    (add_net "Net-(J3-Pad16)")
+    (add_net "Net-(J3-Pad17)")
+    (add_net "Net-(J3-Pad18)")
+    (add_net "Net-(J3-Pad19)")
+    (add_net "Net-(J3-Pad2)")
+    (add_net "Net-(J3-Pad20)")
+    (add_net "Net-(J3-Pad21)")
+    (add_net "Net-(J3-Pad22)")
+    (add_net "Net-(J3-Pad23)")
+    (add_net "Net-(J3-Pad24)")
+    (add_net "Net-(J3-Pad25)")
+    (add_net "Net-(J3-Pad26)")
+    (add_net "Net-(J3-Pad27)")
+    (add_net "Net-(J3-Pad28)")
+    (add_net "Net-(J3-Pad29)")
+    (add_net "Net-(J3-Pad3)")
+    (add_net "Net-(J3-Pad30)")
+    (add_net "Net-(J3-Pad31)")
+    (add_net "Net-(J3-Pad32)")
+    (add_net "Net-(J3-Pad33)")
+    (add_net "Net-(J3-Pad34)")
+    (add_net "Net-(J3-Pad35)")
+    (add_net "Net-(J3-Pad36)")
+    (add_net "Net-(J3-Pad37)")
+    (add_net "Net-(J3-Pad38)")
+    (add_net "Net-(J3-Pad39)")
+    (add_net "Net-(J3-Pad4)")
+    (add_net "Net-(J3-Pad40)")
+    (add_net "Net-(J3-Pad5)")
+    (add_net "Net-(J3-Pad6)")
+    (add_net "Net-(J3-Pad7)")
+    (add_net "Net-(J3-Pad8)")
+    (add_net "Net-(J3-Pad9)")
     (add_net "Net-(U1-Pad14)")
     (add_net "Net-(U1-Pad15)")
@@
     (add_net "Net-(U2-Pad7)")
   )
+  (module Connector_PinSocket_2.54mm:PinSocket_2x20_P2.54mm_Vertical (layer F.Cu)
+    (at 531.241 89.281)
+    (descr "Through hole straight socket strip, 2x20, 2.54mm pitch, double cols (from Kicad 4.0.7), script generated")
+    (tags "Through hole socket strip THT 2x20 2.54mm double row")
+    (fp_text reference J3 (at -1.27 -2.77) (layer F.SilkS)
+      (effects (font (size 1 1) (thickness 0.15)))
+    )
+    (fp_text value Raspberry_Pi_2_3 (at -1.27 51.03) (layer F.Fab)
+      (effects (font (size 1 1) (thickness 0.15)))
+    )
+    (fp_text user %R (at -1.27 24.13 90) (layer F.Fab)
+      (effects (font (size 1 1) (thickness 0.15)))
+    )
+    (fp_line (start -3.81 -1.27) (end 0.27 -1.27) (layer F.Fab) (width 0.1))
+    (fp_line (start 0.27 -1.27) (end 1.27 -0.27) (layer F.Fab) (width 0.1))
+    (fp_line (start 1.27 -0.27) (end 1.27 49.53) (layer F.Fab) (width 0.1))
+    (fp_line (start 1.27 49.53) (end -3.81 49.53) (layer F.Fab) (width 0.1))
+    (fp_line (start -3.81 49.53) (end -3.81 -1.27) (layer F.Fab) (width 0.1))
+    (fp_line (start -3.87 -1.33) (end -1.27 -1.33) (layer F.SilkS) (width 0.12))
+    (fp_line (start -3.87 -1.33) (end -3.87 49.59) (layer F.SilkS) (width 0.12))
+    (fp_line (start -3.87 49.59) (end 1.33 49.59) (layer F.SilkS) (width 0.12))
+    (fp_line (start 1.33 1.27) (end 1.33 49.59) (layer F.SilkS) (width 0.12))
+    (fp_line (start -1.27 1.27) (end 1.33 1.27) (layer F.SilkS) (width 0.12))
+    (fp_line (start -1.27 -1.33) (end -1.27 1.27) (layer F.SilkS) (width 0.12))
+    (fp_line (start 1.33 -1.33) (end 1.33 0) (layer F.SilkS) (width 0.12))
+    (fp_line (start 0 -1.33) (end 1.33 -1.33) (layer F.SilkS) (width 0.12))
+    (fp_line (start -4.34 -1.8) (end 1.76 -1.8) (layer F.CrtYd) (width 0.05))
+    (fp_line (start 1.76 -1.8) (end 1.76 50) (layer F.CrtYd) (width 0.05))
+    (fp_line (start 1.76 50) (end -4.34 50) (layer F.CrtYd) (width 0.05))
+    (fp_line (start -4.34 50) (end -4.34 -1.8) (layer F.CrtYd) (width 0.05))
+    (pad 40 thru_hole oval (at -2.54 48.26) (size 1.7 1.7) (drill 1) (layers *.Cu *.Mask))
+    (pad 39 thru_hole oval (at 0 48.26) (size 1.7 1.7) (drill 1) (layers *.Cu *.Mask))
+    (pad 38 thru_hole oval (at -2.54 45.72) (size 1.7 1.7) (drill 1) (layers *.Cu *.Mask))
+    (pad 37 thru_hole oval (at 0 45.72) (size 1.7 1.7) (drill 1) (layers *.Cu *.Mask))
+    (pad 36 thru_hole oval (at -2.54 43.18) (size 1.7 1.7) (drill 1) (layers *.Cu *.Mask))
+    (pad 35 thru_hole oval (at 0 43.18) (size 1.7 1.7) (drill 1) (layers *.Cu *.Mask))
+    (pad 34 thru_hole oval (at -2.54 40.64) (size 1.7 1.7) (drill 1) (layers *.Cu *.Mask))
+    (pad 33 thru_hole oval (at 0 40.64) (size 1.7 1.7) (drill 1) (layers *.Cu *.Mask))
+    (pad 32 thru_hole oval (at -2.54 38.1) (size 1.7 1.7) (drill 1) (layers *.Cu *.Mask))
+    (pad 31 thru_hole oval (at 0 38.1) (size 1.7 1.7) (drill 1) (layers *.Cu *.Mask))
+    (pad 30 thru_hole oval (at -2.54 35.56) (size 1.7 1.7) (drill 1) (layers *.Cu *.Mask))
+    (pad 29 thru_hole oval (at 0 35.56) (size 1.7 1.7) (drill 1) (layers *.Cu *.Mask))
+    (pad 28 thru_hole oval (at -2.54 33.02) (size 1.7 1.7) (drill 1) (layers *.Cu *.Mask))
+    (pad 27 thru_hole oval (at 0 33.02) (size 1.7 1.7) (drill 1) (layers *.Cu *.Mask))
+    (pad 26 thru_hole oval (at -2.54 30.48) (size 1.7 1.7) (drill 1) (layers *.Cu *.Mask))
+    (pad 25 thru_hole oval (at 0 30.48) (size 1.7 1.7) (drill 1) (layers *.Cu *.Mask))
+    (pad 24 thru_hole oval (at -2.54 27.94) (size 1.7 1.7) (drill 1) (layers *.Cu *.Mask))
+    (pad 23 thru_hole oval (at 0 27.94) (size 1.7 1.7) (drill 1) (layers *.Cu *.Mask))
+    (pad 22 thru_hole oval (at -2.54 25.4) (size 1.7 1.7) (drill 1) (layers *.Cu *.Mask))
+    (pad 21 thru_hole oval (at 0 25.4) (size 1.7 1.7) (drill 1) (layers *.Cu *.Mask))
+    (pad 20 thru_hole oval (at -2.54 22.86) (size 1.7 1.7) (drill 1) (layers *.Cu *.Mask))
+    (pad 19 thru_hole oval (at 0 22.86) (size 1.7 1.7) (drill 1) (layers *.Cu *.Mask))
+    (pad 18 thru_hole oval (at -2.54 20.32) (size 1.7 1.7) (drill 1) (layers *.Cu *.Mask))
+    (pad 17 thru_hole oval (at 0 20.32) (size 1.7 1.7) (drill 1) (layers *.Cu *.Mask))
+    (pad 16 thru_hole oval (at -2.54 17.78) (size 1.7 1.7) (drill 1) (layers *.Cu *.Mask))
+    (pad 15 thru_hole oval (at 0 17.78) (size 1.7 1.7) (drill 1) (layers *.Cu *.Mask))
+    (pad 14 thru_hole oval (at -2.54 15.24) (size 1.7 1.7) (drill 1) (layers *.Cu *.Mask))
+    (pad 13 thru_hole oval (at 0 15.24) (size 1.7 1.7) (drill 1) (layers *.Cu *.Mask))
+    (pad 12 thru_hole oval (at -2.54 12.7) (size 1.7 1.7) (drill 1) (layers *.Cu *.Mask))
+    (pad 11 thru_hole oval (at 0 12.7) (size 1.7 1.7) (drill 1) (layers *.Cu *.Mask))
+    (pad 10 thru_hole oval (at -2.54 10.16) (size 1.7 1.7) (drill 1) (layers *.Cu *.Mask))
+    (pad 9 thru_hole oval (at 0 10.16) (size 1.7 1.7) (drill 1) (layers *.Cu *.Mask))
+    (pad 8 thru_hole oval (at -2.54 7.62) (size 1.7 1.7) (drill 1) (layers *.Cu *.Mask))
+    (pad 7 thru_hole oval (at 0 7.62) (size 1.7 1.7) (drill 1) (layers *.Cu *.Mask))
+    (pad 6 thru_hole oval (at -2.54 5.08) (size 1.7 1.7) (drill 1) (layers *.Cu *.Mask))
+    (pad 5 thru_hole oval (at 0 5.08) (size 1.7 1.7) (drill 1) (layers *.Cu *.Mask))
+    (pad 4 thru_hole oval (at -2.54 2.54) (size 1.7 1.7) (drill 1) (layers *.Cu *.Mask))
+    (pad 3 thru_hole oval (at 0 2.54) (size 1.7 1.7) (drill 1) (layers *.Cu *.Mask))
+    (pad 2 thru_hole oval (at -2.54 0) (size 1.7 1.7) (drill 1) (layers *.Cu *.Mask))
+    (pad 1 thru_hole rect (at 0 0) (size 1.7 1.7) (drill 1) (layers *.Cu *.Mask))
+    (model ${KISYS3DMOD}/Connector_PinSocket_2.54mm.3dshapes/PinSocket_2x20_P2.54mm_Vertical.wrl
+      (at (xyz 0 0 0))
+      (scale (xyz 1 1 1))
+      (rotate (xyz 0 0 0))
+    )
+  )
   (module Connector_PinSocket_2.54mm:PinSocket_2x06_P2.54mm_Horizontal (layer F.Cu)

Commit message: checkpoint
Parts:
- added J4: Screw_Terminal_01x02, TerminalBlock:TerminalBlock_bornier-2_P5.08mm, F.Cu at (315.6, -49.1)
- added J5: Screw_Terminal_01x02, TerminalBlock:TerminalBlock_bornier-2_P5.08mm, F.Cu at (315.6, -58.2)
- added R1: R33, Resistor_SMD:R_0805_2012Metric_Pad1.20x1.40mm_HandSolder, F.Cu at (7.75, 0.51)
- added R10: R33, Resistor_SMD:R_0805_2012Metric_Pad1.20x1.40mm_HandSolder, F.Cu at (151.0, -0.13)
- added R11: R33, Resistor_SMD:R_0805_2012Metric_Pad1.20x1.40mm_HandSolder, F.Cu at (166.9, -0.13)
- added R12: R33, Resistor_SMD:R_0805_2012Metric_Pad1.20x1.40mm_HandSolder, F.Cu at (182.7, -0.13)
- added R13: R33, Resistor_SMD:R_0805_2012Metric_Pad1.20x1.40mm_HandSolder, F.Cu at (198.6, -0.13)
- added R14: R33, Resistor_SMD:R_0805_2012Metric_Pad1.20x1.40mm_HandSolder, F.Cu at (214.5, -0.13)
- added R15: R33, Resistor_SMD:R_0805_2012Metric_Pad1.20x1.40mm_HandSolder, F.Cu at (230.4, -0.13)
- added R16: R33, Resistor_SMD:R_0805_2012Metric_Pad1.20x1.40mm_HandSolder, F.Cu at (246.2, -0.13)
- added R17: R33, Resistor_SMD:R_0805_2012Metric_Pad1.20x1.40mm_HandSolder, F.Cu at (262.1, -0.13)
- added R18: R33, Resistor_SMD:R_0805_2012Metric_Pad1.20x1.40mm_HandSolder, F.Cu at (278.0, -0.13)
- added R19: R33, Resistor_SMD:R_0805_2012Metric_Pad1.20x1.40mm_HandSolder, F.Cu at (293.9, -0.13)
- added R2: R33, Resistor_SMD:R_0805_2012Metric_Pad1.20x1.40mm_HandSolder, F.Cu at (24.0, -0.13)
- added R20: R33, Resistor_SMD:R_0805_2012Metric_Pad1.20x1.40mm_HandSolder, F.Cu at (309.7, -0.13)
- added R21: R33, Resistor_SMD:R_0805_2012Metric_Pad1.20x1.40mm_HandSolder, F.Cu at (325.6, -0.13)
- added R22: R33, Resistor_SMD:R_0805_2012Metric_Pad1.20x1.40mm_HandSolder, F.Cu at (341.5, -0.13)
- added R23: R33, Resistor_SMD:R_0805_2012Metric_Pad1.20x1.40mm_HandSolder, F.Cu at (357.4, -0.13)
- added R24: R33, Resistor_SMD:R_0805_2012Metric_Pad1.20x1.40mm_HandSolder, F.Cu at (373.2, -0.13)
- added R25: R33, Resistor_SMD:R_0805_2012Metric_Pad1.20x1.40mm_HandSolder, F.Cu at (389.1, -0.13)
- added R26: R33, Resistor_SMD:R_0805_2012Metric_Pad1.20x1.40mm_HandSolder, F.Cu at (405.0, -0.13)
- added R27: R33, Resistor_SMD:R_0805_2012Metric_Pad1.20x1.40mm_HandSolder, F.Cu at (420.9, -0.13)
- added R28: R33, Resistor_SMD:R_0805_2012Metric_Pad1.20x1.40mm_HandSolder, F.Cu at (436.7, -0.13)
- added R29: R33, Resistor_SMD:R_0805_2012Metric_Pad1.20x1.40mm_HandSolder, F.Cu at (452.6, -0.13)
- added R3: R33, Resistor_SMD:R_0805_2012Metric_Pad1.20x1.40mm_HandSolder, F.Cu at (39.9, -0.13)
- added R30: R33, Resistor_SMD:R_0805_2012Metric_Pad1.20x1.40mm_HandSolder, F.Cu at (468.5, -0.13)
- added R31: R33, Resistor_SMD:R_0805_2012Metric_Pad1.20x1.40mm_HandSolder, F.Cu at (484.4, -0.13)
- added R32: R33, Resistor_SMD:R_0805_2012Metric_Pad1.20x1.40mm_HandSolder, F.Cu at (500.2, -0.13)
- added R33: R33, Resistor_SMD:R_0805_2012Metric_Pad1.20x1.40mm_HandSolder, F.Cu at (215.3, -28.2)
- added R34: R33, Resistor_SMD:R_0805_2012Metric_Pad1.20x1.40mm_HandSolder, F.Cu at (221.1, -28.2)
- added R35: R33, Resistor_SMD:R_0805_2012Metric_Pad1.20x1.40mm_HandSolder, F.Cu at (226.9, -28.2)
- added R36: R33, Resistor_SMD:R_0805_2012Metric_Pad1.20x1.40mm_HandSolder, F.Cu at (232.7, -28.2)
- added R37: R33, Resistor_SMD:R_0805_2012Metric_Pad1.20x1.40mm_HandSolder, F.Cu at (238.5, -28.2)
- added R38: R33, Resistor_SMD:R_0805_2012Metric_Pad1.20x1.40mm_HandSolder, F.Cu at (244.4, -28.2)
- added R39: R33, Resistor_SMD:R_0805_2012Metric_Pad1.20x1.40mm_HandSolder, F.Cu at (250.2, -28.2)
- added R4: R33, Resistor_SMD:R_0805_2012Metric_Pad1.20x1.40mm_HandSolder, F.Cu at (55.8, -0.13)
- added R40: R33, Resistor_SMD:R_0805_2012Metric_Pad1.20x1.40mm_HandSolder, F.Cu at (256.0, -28.2)
- added R41: R33, Resistor_SMD:R_0805_2012Metric_Pad1.20x1.40mm_HandSolder, F.Cu at (261.8, -28.2)
- added R42: R33, Resistor_SMD:R_0805_2012Metric_Pad1.20x1.40mm_HandSolder, F.Cu at (267.6, -28.2)
- added R43: R33, Resistor_SMD:R_0805_2012Metric_Pad1.20x1.40mm_HandSolder, F.Cu at (273.4, -28.2)
- added R44: R33, Resistor_SMD:R_0805_2012Metric_Pad1.20x1.40mm_HandSolder, F.Cu at (279.3, -28.2)
- added R45: R33, Resistor_SMD:R_0805_2012Metric_Pad1.20x1.40mm_HandSolder, F.Cu at (285.1, -28.2)
- added R46: R33, Resistor_SMD:R_0805_2012Metric_Pad1.20x1.40mm_HandSolder, F.Cu at (290.9, -28.2)
- added R47: R33, Resistor_SMD:R_0805_2012Metric_Pad1.20x1.40mm_HandSolder, F.Cu at (296.7, -28.2)
- added R48: R33, Resistor_SMD:R_0805_2012Metric_Pad1.20x1.40mm_HandSolder, F.Cu at (302.5, -28.2)
- added R49: R33, Resistor_SMD:R_0805_2012Metric_Pad1.20x1.40mm_HandSolder, F.Cu at (308.3, -28.2)
- added R5: R33, Resistor_SMD:R_0805_2012Metric_Pad1.20x1.40mm_HandSolder, F.Cu at (71.6, -0.13)
- added R50: R33, Resistor_SMD:R_0805_2012Metric_Pad1.20x1.40mm_HandSolder, F.Cu at (314.2, -28.2)
- added R51: R33, Resistor_SMD:R_0805_2012Metric_Pad1.20x1.40mm_HandSolder, F.Cu at (320.0, -28.2)
- added R52: R33, Resistor_SMD:R_0805_2012Metric_Pad1.20x1.40mm_HandSolder, F.Cu at (325.8, -28.2)
- added R53: R33, Resistor_SMD:R_0805_2012Metric_Pad1.20x1.40mm_HandSolder, F.Cu at (331.6, -28.2)
- added R54: R33, Resistor_SMD:R_0805_2012Metric_Pad1.20x1.40mm_HandSolder, F.Cu at (337.4, -28.2)
- added R55: R33, Resistor_SMD:R_0805_2012Metric_Pad1.20x1.40mm_HandSolder, F.Cu at (343.2, -28.2)
- added R56: R33, Resistor_SMD:R_0805_2012Metric_Pad1.20x1.40mm_HandSolder, F.Cu at (349.1, -28.2)
- added R57: R33, Resistor_SMD:R_0805_2012Metric_Pad1.20x1.40mm_HandSolder, F.Cu at (354.9, -28.2)
- added R58: R33, Resistor_SMD:R_0805_2012Metric_Pad1.20x1.40mm_HandSolder, F.Cu at (360.7, -28.2)
- added R59: R33, Resistor_SMD:R_0805_2012Metric_Pad1.20x1.40mm_HandSolder, F.Cu at (366.5, -28.2)
- added R6: R33, Resistor_SMD:R_0805_2012Metric_Pad1.20x1.40mm_HandSolder, F.Cu at (87.5, -0.13)
- added R60: R33, Resistor_SMD:R_0805_2012Metric_Pad1.20x1.40mm_HandSolder, F.Cu at (372.3, -28.2)
- added R61: R33, Resistor_SMD:R_0805_2012Metric_Pad1.20x1.40mm_HandSolder, F.Cu at (378.2, -28.2)
- added R62: R33, Resistor_SMD:R_0805_2012Metric_Pad1.20x1.40mm_HandSolder, F.Cu at (384.0, -28.2)
- added R63: R33, Resistor_SMD:R_0805_2012Metric_Pad1.20x1.40mm_HandSolder, F.Cu at (389.8, -28.2)
- added R64: R33, Resistor_SMD:R_0805_2012Metric_Pad1.20x1.40mm_HandSolder, F.Cu at (395.6, -28.2)
- added R7: R33, Resistor_SMD:R_0805_2012Metric_Pad1.20x1.40mm_HandSolder, F.Cu at (103.4, -0.13)
- added R8: R33, Resistor_SMD:R_0805_2012Metric_Pad1.20x1.40mm_HandSolder, F.Cu at (119.2, -0.13)
- added R9: R33, Resistor_SMD:R_0805_2012Metric_Pad1.20x1.40mm_HandSolder, F.Cu at (135.1, -0.13)
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Connections:
- D00A1 pad 2: /row0 -> Net-(D00A1-Pad2)
- D00A2 pad 2: /row32 -> Net-(D00A2-Pad2)
- D00B1 pad 2: /row0 -> Net-(D00A1-Pad2)
- D00B2 pad 2: /row32 -> Net-(D00A2-Pad2)
- D00C1 pad 2: /row0 -> Net-(D00A1-Pad2)
- D00C2 pad 2: /row32 -> Net-(D00A2-Pad2)
- D00D1 pad 2: /row0 -> Net-(D00A1-Pad2)
- D00D2 pad 2: /row32 -> Net-(D00A2-Pad2)
- D00E1 pad 2: /row0 -> Net-(D00A1-Pad2)
- D00E2 pad 2: /row32 -> Net-(D00A2-Pad2)
- D00F1 pad 2: /row0 -> Net-(D00A1-Pad2)
- D00F2 pad 2: /row32 -> Net-(D00A2-Pad2)
- D00G1 pad 2: /row0 -> Net-(D00A1-Pad2)
- D00G2 pad 2: /row32 -> Net-(D00A2-Pad2)
- D00H1 pad 2: /row0 -> Net-(D00A1-Pad2)
- D00H2 pad 2: /row32 -> Net-(D00A2-Pad2)
- D01A1 pad 2: /row1 -> Net-(D01A1-Pad2)
- D01A2 pad 2: /row33 -> Net-(D01A2-Pad2)
- D01B1 pad 2: /row1 -> Net-(D01A1-Pad2)
- D01B2 pad 2: /row33 -> Net-(D01A2-Pad2)
- D01C1 pad 2: /row1 -> Net-(D01A1-Pad2)
- D01C2 pad 2: /row33 -> Net-(D01A2-Pad2)
- D01D1 pad 2: /row1 -> Net-(D01A1-Pad2)
- D01D2 pad 2: /row33 -> Net-(D01A2-Pad2)
- D01E1 pad 2: /row1 -> Net-(D01A1-Pad2)
- D01E2 pad 2: /row33 -> Net-(D01A2-Pad2)
- D01F1 pad 2: /row1 -> Net-(D01A1-Pad2)
- D01F2 pad 2: /row33 -> Net-(D01A2-Pad2)
- D01G1 pad 2: /row1 -> Net-(D01A1-Pad2)
- D01G2 pad 2: /row33 -> Net-(D01A2-Pad2)
- D01H1 pad 2: /row1 -> Net-(D01A1-Pad2)
- D01H2 pad 2: /row33 -> Net-(D01A2-Pad2)
- D02A1 pad 2: /row2 -> Net-(D02A1-Pad2)
- D02A2 pad 2: /row34 -> Net-(D02A2-Pad2)
- D02B1 pad 2: /row2 -> Net-(D02A1-Pad2)
- D02B2 pad 2: /row34 -> Net-(D02A2-Pad2)
- D02C1 pad 2: /row2 -> Net-(D02A1-Pad2)
- D02C2 pad 2: /row34 -> Net-(D02A2-Pad2)
- D02D1 pad 2: /row2 -> Net-(D02A1-Pad2)
- D02D2 pad 2: /row34 -> Net-(D02A2-Pad2)
- D02E1 pad 2: /row2 -> Net-(D02A1-Pad2)
- D02E2 pad 2: /row34 -> Net-(D02A2-Pad2)
- D02F1 pad 2: /row2 -> Net-(D02A1-Pad2)
- D02F2 pad 2: /row34 -> Net-(D02A2-Pad2)
- D02G1 pad 2: /row2 -> Net-(D02A1-Pad2)
- D02G2 pad 2: /row34 -> Net-(D02A2-Pad2)
- D02H1 pad 2: /row2 -> Net-(D02A1-Pad2)
- D02H2 pad 2: /row34 -> Net-(D02A2-Pad2)
- D03A1 pad 2: /row3 -> Net-(D03A1-Pad2)
- D03A2 pad 2: /row35 -> Net-(D03A2-Pad2)
- D03B1 pad 2: /row3 -> Net-(D03A1-Pad2)
- D03B2 pad 2: /row35 -> Net-(D03A2-Pad2)
- D03C1 pad 2: /row3 -> Net-(D03A1-Pad2)
- D03C2 pad 2: /row35 -> Net-(D03A2-Pad2)
- D03D1 pad 2: /row3 -> Net-(D03A1-Pad2)
- D03D2 pad 2: /row35 -> Net-(D03A2-Pad2)
- D03E1 pad 2: /row3 -> Net-(D03A1-Pad2)
- D03E2 pad 2: /row35 -> Net-(D03A2-Pad2)
- D03F1 pad 2: /row3 -> Net-(D03A1-Pad2)
- D03F2 pad 2: /row35 -> Net-(D03A2-Pad2)
- D03G1 pad 2: /row3 -> Net-(D03A1-Pad2)
- D03G2 pad 2: /row35 -> Net-(D03A2-Pad2)
- D03H1 pad 2: /row3 -> Net-(D03A1-Pad2)
- D03H2 pad 2: /row35 -> Net-(D03A2-Pad2)
- D04A1 pad 2: /row4 -> Net-(D04A1-Pad2)
- D04A2 pad 2: /row36 -> Net-(D04A2-Pad2)
- D04B1 pad 2: /row4 -> Net-(D04A1-Pad2)
- D04B2 pad 2: /row36 -> Net-(D04A2-Pad2)
- D04C1 pad 2: /row4 -> Net-(D04A1-Pad2)
- D04C2 pad 2: /row36 -> Net-(D04A2-Pad2)
- D04D1 pad 2: /row4 -> Net-(D04A1-Pad2)
- D04D2 pad 2: /row36 -> Net-(D04A2-Pad2)
- D04E1 pad 2: /row4 -> Net-(D04A1-Pad2)
- D04E2 pad 2: /row36 -> Net-(D04A2-Pad2)
- D04F1 pad 2: /row4 -> Net-(D04A1-Pad2)
- D04F2 pad 2: /row36 -> Net-(D04A2-Pad2)
- D04G1 pad 2: /row4 -> Net-(D04A1-Pad2)
- D04G2 pad 2: /row36 -> Net-(D04A2-Pad2)
- D04H1 pad 2: /row4 -> Net-(D04A1-Pad2)
- D04H2 pad 2: /row36 -> Net-(D04A2-Pad2)
- D05A1 pad 2: /row5 -> Net-(D05A1-Pad2)
- D05A2 pad 2: /row37 -> Net-(D05A2-Pad2)
- D05B1 pad 2: /row5 -> Net-(D05A1-Pad2)
- D05B2 pad 2: /row37 -> Net-(D05A2-Pad2)
- D05C1 pad 2: /row5 -> Net-(D05A1-Pad2)
- D05C2 pad 2: /row37 -> Net-(D05A2-Pad2)
- D05D1 pad 2: /row5 -> Net-(D05A1-Pad2)
- D05D2 pad 2: /row37 -> Net-(D05A2-Pad2)
- D05E1 pad 2: /row5 -> Net-(D05A1-Pad2)
- D05E2 pad 2: /row37 -> Net-(D05A2-Pad2)
- D05F1 pad 2: /row5 -> Net-(D05A1-Pad2)
- D05F2 pad 2: /row37 -> Net-(D05A2-Pad2)
- D05G1 pad 2: /row5 -> Net-(D05A1-Pad2)
- D05G2 pad 2: /row37 -> Net-(D05A2-Pad2)
- D05H1 pad 2: /row5 -> Net-(D05A1-Pad2)
- D05H2 pad 2: /row37 -> Net-(D05A2-Pad2)
- D06A1 pad 2: /row6 -> Net-(D06A1-Pad2)
- D06A2 pad 2: /row38 -> Net-(D06A2-Pad2)
- D06B1 pad 2: /row6 -> Net-(D06A1-Pad2)
- D06B2 pad 2: /row38 -> Net-(D06A2-Pad2)
- D06C1 pad 2: /row6 -> Net-(D06A1-Pad2)
- D06C2 pad 2: /row38 -> Net-(D06A2-Pad2)
- D06D1 pad 2: /row6 -> Net-(D06A1-Pad2)
- D06D2 pad 2: /row38 -> Net-(D06A2-Pad2)
- D06E1 pad 2: /row6 -> Net-(D06A1-Pad2)
- D06E2 pad 2: /row38 -> Net-(D06A2-Pad2)
- D06F1 pad 2: /row6 -> Net-(D06A1-Pad2)
- D06F2 pad 2: /row38 -> Net-(D06A2-Pad2)
- D06G1 pad 2: /row6 -> Net-(D06A1-Pad2)
- D06G2 pad 2: /row38 -> Net-(D06A2-Pad2)
- D06H1 pad 2: /row6 -> Net-(D06A1-Pad2)
- D06H2 pad 2: /row38 -> Net-(D06A2-Pad2)
- D07A1 pad 2: /row7 -> Net-(D07A1-Pad2)
- D07A2 pad 2: /row39 -> Net-(D07A2-Pad2)
- D07B1 pad 2: /row7 -> Net-(D07A1-Pad2)
- D07B2 pad 2: /row39 -> Net-(D07A2-Pad2)
- D07C1 pad 2: /row7 -> Net-(D07A1-Pad2)
- D07C2 pad 2: /row39 -> Net-(D07A2-Pad2)
- D07D1 pad 2: /row7 -> Net-(D07A1-Pad2)
- D07D2 pad 2: /row39 -> Net-(D07A2-Pad2)
- D07E1 pad 2: /row7 -> Net-(D07A1-Pad2)
- D07E2 pad 2: /row39 -> Net-(D07A2-Pad2)
- D07F1 pad 2: /row7 -> Net-(D07A1-Pad2)
- D07F2 pad 2: /row39 -> Net-(D07A2-Pad2)
- D07G1 pad 2: /row7 -> Net-(D07A1-Pad2)
- D07G2 pad 2: /row39 -> Net-(D07A2-Pad2)
- D07H1 pad 2: /row7 -> Net-(D07A1-Pad2)
- D07H2 pad 2: /row39 -> Net-(D07A2-Pad2)
- D08A1 pad 2: /row8 -> Net-(D08A1-Pad2)
- D08A2 pad 2: /row40 -> Net-(D08A2-Pad2)
- D08B1 pad 2: /row8 -> Net-(D08A1-Pad2)
- D08B2 pad 2: /row40 -> Net-(D08A2-Pad2)
- D08C1 pad 2: /row8 -> Net-(D08A1-Pad2)
- D08C2 pad 2: /row40 -> Net-(D08A2-Pad2)
- D08D1 pad 2: /row8 -> Net-(D08A1-Pad2)
- D08D2 pad 2: /row40 -> Net-(D08A2-Pad2)
- D08E1 pad 2: /row8 -> Net-(D08A1-Pad2)
- D08E2 pad 2: /row40 -> Net-(D08A2-Pad2)
- D08F1 pad 2: /row8 -> Net-(D08A1-Pad2)
- D08F2 pad 2: /row40 -> Net-(D08A2-Pad2)
- D08G1 pad 2: /row8 -> Net-(D08A1-Pad2)
- D08G2 pad 2: /row40 -> Net-(D08A2-Pad2)
- D08H1 pad 2: /row8 -> Net-(D08A1-Pad2)
- D08H2 pad 2: /row40 -> Net-(D08A2-Pad2)
- D09A1 pad 2: /row9 -> Net-(D09A1-Pad2)
- D09A2 pad 2: /row41 -> Net-(D09A2-Pad2)
- D09B1 pad 2: /row9 -> Net-(D09A1-Pad2)
- D09B2 pad 2: /row41 -> Net-(D09A2-Pad2)
- D09C1 pad 2: /row9 -> Net-(D09A1-Pad2)
- D09C2 pad 2: /row41 -> Net-(D09A2-Pad2)
- D09D1 pad 2: /row9 -> Net-(D09A1-Pad2)
- D09D2 pad 2: /row41 -> Net-(D09A2-Pad2)
- D09E1 pad 2: /row9 -> Net-(D09A1-Pad2)
- D09E2 pad 2: /row41 -> Net-(D09A2-Pad2)
- D09F1 pad 2: /row9 -> Net-(D09A1-Pad2)
- D09F2 pad 2: /row41 -> Net-(D09A2-Pad2)
- D09G1 pad 2: /row9 -> Net-(D09A1-Pad2)
- D09G2 pad 2: /row41 -> Net-(D09A2-Pad2)
- D09H1 pad 2: /row9 -> Net-(D09A1-Pad2)
- D09H2 pad 2: /row41 -> Net-(D09A2-Pad2)
- D10A1 pad 2: /row10 -> Net-(D10A1-Pad2)
- D10A2 pad 2: /row42 -> Net-(D10A2-Pad2)
- D10B1 pad 2: /row10 -> Net-(D10A1-Pad2)
- D10B2 pad 2: /row42 -> Net-(D10A2-Pad2)
- D10C1 pad 2: /row10 -> Net-(D10A1-Pad2)
- D10C2 pad 2: /row42 -> Net-(D10A2-Pad2)
- D10D1 pad 2: /row10 -> Net-(D10A1-Pad2)
- D10D2 pad 2: /row42 -> Net-(D10A2-Pad2)
- D10E1 pad 2: /row10 -> Net-(D10A1-Pad2)
- D10E2 pad 2: /row42 -> Net-(D10A2-Pad2)
- D10F1 pad 2: /row10 -> Net-(D10A1-Pad2)
- D10F2 pad 2: /row42 -> Net-(D10A2-Pad2)
- D10G1 pad 2: /row10 -> Net-(D10A1-Pad2)
- D10G2 pad 2: /row42 -> Net-(D10A2-Pad2)
- D10H1 pad 2: /row10 -> Net-(D10A1-Pad2)
- D10H2 pad 2: /row42 -> Net-(D10A2-Pad2)
- D11A1 pad 2: /row11 -> Net-(D11A1-Pad2)
- D11A2 pad 2: /row43 -> Net-(D11A2-Pad2)
- D11B1 pad 2: /row11 -> Net-(D11A1-Pad2)
- D11B2 pad 2: /row43 -> Net-(D11A2-Pad2)
- D11C1 pad 2: /row11 -> Net-(D11A1-Pad2)
- D11C2 pad 2: /row43 -> Net-(D11A2-Pad2)
- D11D1 pad 2: /row11 -> Net-(D11A1-Pad2)
- D11D2 pad 2: /row43 -> Net-(D11A2-Pad2)
- D11E1 pad 2: /row11 -> Net-(D11A1-Pad2)
- D11E2 pad 2: /row43 -> Net-(D11A2-Pad2)
- D11F1 pad 2: /row11 -> Net-(D11A1-Pad2)
- D11F2 pad 2: /row43 -> Net-(D11A2-Pad2)
- D11G1 pad 2: /row11 -> Net-(D11A1-Pad2)
- D11G2 pad 2: /row43 -> Net-(D11A2-Pad2)
- D11H1 pad 2: /row11 -> Net-(D11A1-Pad2)
- D11H2 pad 2: /row43 -> Net-(D11A2-Pad2)
- D12A1 pad 2: /row12 -> Net-(D12A1-Pad2)
- D12A2 pad 2: /row44 -> Net-(D12A2-Pad2)
- D12B1 pad 2: /row12 -> Net-(D12A1-Pad2)
- D12B2 pad 2: /row44 -> Net-(D12A2-Pad2)
- D12C1 pad 2: /row12 -> Net-(D12A1-Pad2)
- D12C2 pad 2: /row44 -> Net-(D12A2-Pad2)
- D12D1 pad 2: /row12 -> Net-(D12A1-Pad2)
- D12D2 pad 2: /row44 -> Net-(D12A2-Pad2)
- D12E1 pad 2: /row12 -> Net-(D12A1-Pad2)
- D12E2 pad 2: /row44 -> Net-(D12A2-Pad2)
- D12F1 pad 2: /row12 -> Net-(D12A1-Pad2)
- D12F2 pad 2: /row44 -> Net-(D12A2-Pad2)
- D12G1 pad 2: /row12 -> Net-(D12A1-Pad2)
- D12G2 pad 2: /row44 -> Net-(D12A2-Pad2)
- D12H1 pad 2: /row12 -> Net-(D12A1-Pad2)
- D12H2 pad 2: /row44 -> Net-(D12A2-Pad2)
- D13A1 pad 2: /row13 -> Net-(D13A1-Pad2)
- D13A2 pad 2: /row45 -> Net-(D13A2-Pad2)
- D13B1 pad 2: /row13 -> Net-(D13A1-Pad2)
- D13B2 pad 2: /row45 -> Net-(D13A2-Pad2)
- D13C1 pad 2: /row13 -> Net-(D13A1-Pad2)
- D13C2 pad 2: /row45 -> Net-(D13A2-Pad2)
- D13D1 pad 2: /row13 -> Net-(D13A1-Pad2)
- D13D2 pad 2: /row45 -> Net-(D13A2-Pad2)
- D13E1 pad 2: /row13 -> Net-(D13A1-Pad2)
- D13E2 pad 2: /row45 -> Net-(D13A2-Pad2)
- D13F1 pad 2: /row13 -> Net-(D13A1-Pad2)
- D13F2 pad 2: /row45 -> Net-(D13A2-Pad2)
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Routing:
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Other:
- net class longrun added: clearance 0.2, trace_width 0.5, via_dia 0.8, via_drill 0.4
