File: cm2.kicad_pcb (KiCad board)
At the start: 2 copper layers, 583 parts, among them J1 Conn_02x06_Counter_Clockwise, J2 Conn_02x06_Counter_Clockwise, J3 Raspberry_Pi_2_3, J4 Screw_Terminal_01x02, J5 Screw_Terminal_01x02, U1 HT1632C-52LQFP, U2 HT1632C-52LQFP

Commit message: checkpoint
Parts:
- added C1: 100uF, Capacitor_THT:CP_Radial_D8.0mm_P5.00mm, F.Cu at (-41.7, -2.79)
- added C2: 100uF, Capacitor_THT:CP_Radial_D8.0mm_P5.00mm, F.Cu at (-43.4, 240.2)
- added C3: 10uF, Capacitor_SMD:C_1206_3216Metric_Pad1.33x1.80mm_HandSolder, F.Cu at (-37.6, 193.0)
- added C4: 10uF, Capacitor_SMD:C_1206_3216Metric_Pad1.33x1.80mm_HandSolder, F.Cu at (-36.6, 222.6)
- added C5: 10uF, Capacitor_SMD:C_1206_3216Metric_Pad1.33x1.80mm_HandSolder, F.Cu at (-36.3, 21.0)
- added C6: 10uF, Capacitor_SMD:C_1206_3216Metric_Pad1.33x1.80mm_HandSolder, F.Cu at (-38.5, 49.0)
- added J6: Conn_02x06_Counter_Clockwise, Connector_PinHeader_2.54mm:PinHeader_2x06_P2.54mm_Horizontal, F.Cu at (-29.1, -2.16)
- added J7: Conn_02x06_Counter_Clockwise, Connector_PinSocket_2.54mm:PinSocket_2x06_P2.54mm_Horizontal, F.Cu at (-28.7, 245.6)
- added REF**: MountingHole_3.2mm_M3, MountingHole:MountingHole_3.2mm_M3, F.Cu at (505.8, 120.9)
- added REF**: MountingHole_3.2mm_M3, MountingHole:MountingHole_3.2mm_M3, F.Cu at (504.8, 230.9)
- added REF**: MountingHole_3.2mm_M3, MountingHole:MountingHole_3.2mm_M3, F.Cu at (505.8, 0.00)
- added REF**: MountingHole_3.2mm_M3, MountingHole:MountingHole_3.2mm_M3, F.Cu at (-8.13, 118.9)
- added REF**: MountingHole_3.2mm_M3, MountingHole:MountingHole_3.2mm_M3, F.Cu at (-9.14, 228.9)
- added REF**: MountingHole_3.2mm_M3, MountingHole:MountingHole_3.2mm_M3, F.Cu at (-8.13, -2.03)
- moved J3 582.5 mm to (-51.2, 99.9)
- moved U2 571.1 mm to (-37.6, 208.2)
- moved J5 471.1 mm to (-51.9, 236.5), turned to 270 degrees
- moved J4 367.6 mm to (-49.0, -2.67), turned to 270 degrees
- moved R33 337.5 mm to (-0.13, 231.6)
- moved R34 337.5 mm to (5.69, 231.6)
- moved R35 337.5 mm to (11.5, 231.6)
- moved R36 337.5 mm to (17.3, 231.6)
- moved R37 337.5 mm to (23.1, 231.6)
- moved R38 337.5 mm to (29.0, 231.6)
- moved R39 337.5 mm to (34.8, 231.6)
- moved R40 337.5 mm to (40.6, 231.6)
- moved R41 337.5 mm to (46.4, 231.6)
- moved R42 337.5 mm to (52.2, 231.6)
- moved R43 337.5 mm to (58.0, 231.6)
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Connections:
- J3 pad 14: (no net) -> GND
- J3 pad 2: (no net) -> +5V
- J3 pad 4: (no net) -> +5V
- J3 pad 6: (no net) -> GND
- J3 pad 9: (no net) -> GND
- J4 pad 1: (no net) -> GND
- J4 pad 2: (no net) -> +5V
- J5 pad 1: (no net) -> GND
- J5 pad 2: (no net) -> +5V
- U1 pad 14: Net-(U1-Pad14) -> GND
- U1 pad 21: (no net) -> +5V
- U1 pad 25: Net-(U1-Pad14) -> GND
- U1 pad 36: Net-(U1-Pad14) -> GND
- U1 pad 38: (no net) -> +5V
- U1 pad 7: (no net) -> +5V
- U2 pad 14: Net-(U2-Pad14) -> GND
- U2 pad 25: Net-(U2-Pad14) -> GND
- U2 pad 36: Net-(U2-Pad14) -> GND
Routing:
- net /col03: track 0.00 -> 695.5 mm, vias 0 -> 1
- net /col01: track 0.00 -> 612.1 mm, vias 0 -> 1
- net /row19: track 0.00 -> 344.9 mm
- net /row18: track 0.00 -> 327.0 mm
- net /col02: track 0.00 -> 317.0 mm, vias 0 -> 1
- net /row17: track 0.00 -> 309.2 mm
- net /col07: track 0.00 -> 304.6 mm, vias 0 -> 1
- net /row16: track 0.00 -> 292.1 mm
- net /row15: track 0.00 -> 274.9 mm
- net /col06: track 0.00 -> 266.3 mm, vias 0 -> 1
- net /row14: track 0.00 -> 257.7 mm
- net /row13: track 0.00 -> 240.6 mm
- net /col05: track 0.00 -> 228.7 mm, vias 0 -> 1
- net /row12: track 0.00 -> 223.2 mm
- net /row11: track 0.00 -> 206.6 mm
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- added copper zone on F.Cu, net +5V
- added copper zone on B.Cu, net GND

Commit message: checkpoint
Parts:
- moved R25 62.5 mm to (388.0, 48.9)
- moved R26 62.5 mm to (403.8, 48.9)
- moved R27 46.7 mm to (419.9, 64.6)
- moved R28 46.6 mm to (435.5, 64.8)
- moved R29 46.6 mm to (451.3, 64.8)
- moved R30 46.6 mm to (467.2, 64.8)
- moved R31 46.6 mm to (483.1, 64.8)
- moved R22 46.6 mm to (340.2, 48.6)
- moved R23 46.6 mm to (356.1, 48.6)
- moved R24 46.6 mm to (372.0, 48.6)
- moved R32 41.7 mm to (494.7, 70.0)
- moved R21 15.9 mm to (324.5, 48.8)
- moved C5 0.85 mm to (-35.6, 21.3), turned to 0 degrees
- turned C6 to 180 degrees
Routing:
- net /col04: track 190.5 -> 781.7 mm
- net /col05: track 228.7 -> 813.3 mm
- net /col07: track 304.6 -> 879.5 mm
- net /col06: track 266.3 -> 839.4 mm
- net /row31: track 0.00 -> 572.5 mm
- net /row30: track 0.00 -> 559.4 mm
- net /row29: track 0.00 -> 539.8 mm
- net /row28: track 0.00 -> 520.2 mm
- net /row27: track 0.00 -> 500.7 mm
- net /row26: track 0.00 -> 479.7 mm
- net /row25: track 0.00 -> 446.8 mm
- net /row24: track 0.00 -> 427.1 mm
- net /row23: track 0.00 -> 410.5 mm
- net /row22: track 0.00 -> 392.6 mm
- net /row21: track 0.00 -> 375.3 mm
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Other:
- net class colbus added: clearance 0.2, trace_width 1, via_dia 0.8, via_drill 0.4

Commit message: checkpoint
Routing:
- net +5V: track 78.3 -> 80.8 mm
Changed lines of the file:
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@@
     (thickness 1.6)
     (drawings 4)
-    (tracks 1115)
+    (tracks 1119)
     (zones 0)
     (modules 597)
@@
   )
   (setup
-    (last_trace_width 1)
+    (last_trace_width 0.5)
     (user_trace_width 0.25)
     (user_trace_width 0.5)
@@
   (segment (start 108.966 108.966) (end 108.966 2.158988) (width 1) (layer B.Cu) (net 40))
   (segment (start 108.966 2.158988) (end 108.839 2.031988) (width 1) (layer B.Cu) (net 40))
-  (segment (start -38.989 2.032) (end 108.839 2.032) (width 1) (layer F.Cu) (net 40))
-  (segment (start -52.197 15.24) (end -38.989 2.032) (width 1) (layer F.Cu) (net 40))
+  (segment (start 108.458 2.413) (end 108.839 2.032) (width 1) (layer F.Cu) (net 40))
+  (segment (start -39.37 2.413) (end 108.458 2.413) (width 1) (layer F.Cu) (net 40))
+  (segment (start -52.197 15.24) (end -39.37 2.413) (width 1) (layer F.Cu) (net 40))
   (segment (start 2.54 15.875) (end 2.54 31.75) (width 1) (layer B.Cu) (net 81) (status 30))
   (segment (start 2.54 31.75) (end 2.54 47.625) (width 0.75) (layer B.Cu) (net 81) (status 30))
@@
   (segment (start -41.656 29.354213) (end -40.678151 30.332062) (width 0.5) (layer F.Cu) (net 146) (status 20))
   (segment (start -41.656 24.003) (end -41.656 29.354213) (width 0.5) (layer F.Cu) (net 146))
-  (segment (start -39.497 26.035) (end -41.529 24.003) (width 1) (layer B.Cu) (net 146))
-  (segment (start -39.497 32.131) (end -39.497 26.035) (width 1) (layer B.Cu) (net 146))
   (segment (start -41.529 9.906) (end -49.022 2.413) (width 1) (layer B.Cu) (net 146))
   (segment (start -41.529 24.003) (end -41.529 9.906) (width 1) (layer B.Cu) (net 146))
@@
   (segment (start -39.497 44.069) (end -37.084 46.482) (width 1) (layer B.Cu) (net 146))
   (segment (start -39.497 32.131) (end -39.497 44.069) (width 1) (layer B.Cu) (net 146))
+  (segment (start -39.497 32.131) (end -41.783 29.845) (width 1) (layer B.Cu) (net 146))
+  (segment (start -41.783 24.257) (end -41.529 24.003) (width 1) (layer B.Cu) (net 146))
+  (segment (start -41.783 29.845) (end -41.783 24.257) (width 1) (layer B.Cu) (net 146))
+  (segment (start -39.497 31.513213) (end -40.678151 30.332062) (width 0.5) (layer F.Cu) (net 146))
+  (segment (start -39.497 32.131) (end -39.497 31.513213) (width 0.5) (layer F.Cu) (net 146))
   (zone (net 145) (net_name GND) (layer B.Cu) (hatch edge 0.508)
     (priority 1)
