File: pcb/cm2.kicad_pcb (KiCad board)
At the start: 2 copper layers, 571.1 x 254 mm, 615 parts, among them J1 top left, J2 bottom left, J3 Raspberry_Pi_2_3, J4 Screw_Terminal_01x02, J5 Screw_Terminal_01x02, U1 HT1632C-52LQFP, U2 HT1632C-52LQFP

Commit message: update to v6.0
Routing:
- net unconnected-(D31G1-Pad2): track 0.00 -> 117.2 mm
- net unconnected-(D31E1-Pad2): track 117.2 -> 0.00 mm
- net unconnected-(R64-Pad2): track 0.00 -> 116.3 mm
- net unconnected-(D31C2-Pad2): track 116.3 -> 0.00 mm
- net unconnected-(D10D1-Pad2): track 0.00 -> 116.3 mm
- net unconnected-(D10A1-Pad2): track 116.3 -> 0.00 mm
- net unconnected-(R28-Pad2): track 116.1 -> 0.00 mm
- net unconnected-(D27B1-Pad2): track 0.00 -> 116.1 mm
- net unconnected-(D08G1-Pad2): track 0.00 -> 116.0 mm
- net unconnected-(D08A1-Pad2): track 116.0 -> 0.00 mm
- net unconnected-(D29H1-Pad2): track 116.0 -> 0.00 mm
- net unconnected-(D29A1-Pad2): track 0.00 -> 116.0 mm
- net unconnected-(D00D2-Pad2): track 0.00 -> 116.0 mm
- net unconnected-(D00A2-Pad2): track 116.0 -> 0.00 mm
- net unconnected-(D01D1-Pad2): track 115.8 -> 0.00 mm
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
Commit message: fix errors from v6 conversion
Parts:
- added C1: 100uF, Capacitor_THT:CP_Radial_D6.3mm_P2.50mm, F.Cu at (10.2, -20.3)
- added C11: 100uF, Capacitor_SMD:CP_Elec_6.3x7.7, F.Cu at (2.12, -20.2)
- added C12: 100uF, Capacitor_SMD:CP_Elec_6.3x7.7, F.Cu at (2.12, -12.0)
- added C2: 100uF, Capacitor_THT:CP_Radial_D6.3mm_P2.50mm, F.Cu at (10.2, -12.5)
Connections:
- net /col00 renamed /col0
- net /col01 renamed /col1
- net /col02 renamed /col2
- net /col03 renamed /col3
- net /col04 renamed /col4
- net /col05 renamed /col5
- net /col06 renamed /col6
- net /col07 renamed /col7
- net /col08 renamed /col8
- net /col09 renamed /col9
- D00A1 pad 2: unconnected-(D00A1-Pad2) -> Net-(D00B1-Pad2)
- D00A2 pad 2: unconnected-(D00A2-Pad2) -> Net-(D00F2-Pad2)
- D00B1 pad 2: unconnected-(D00B1-Pad2) -> Net-(D00B1-Pad2)
- D00B2 pad 2: unconnected-(D00B2-Pad2) -> Net-(D00F2-Pad2)
- D00C1 pad 2: unconnected-(D00C1-Pad2) -> Net-(D00B1-Pad2)
- D00C2 pad 2: unconnected-(D00C2-Pad2) -> Net-(D00F2-Pad2)
- D00D1 pad 2: unconnected-(D00D1-Pad2) -> Net-(D00B1-Pad2)
- D00D2 pad 2: unconnected-(D00D2-Pad2) -> Net-(D00F2-Pad2)
- D00E1 pad 2: unconnected-(D00E1-Pad2) -> Net-(D00B1-Pad2)
- D00E2 pad 2: unconnected-(D00E2-Pad2) -> Net-(D00F2-Pad2)
- D00F1 pad 2: unconnected-(D00F1-Pad2) -> Net-(D00B1-Pad2)
- D00F2 pad 2: unconnected-(D00F2-Pad2) -> Net-(D00F2-Pad2)
- D00G1 pad 2: unconnected-(D00G1-Pad2) -> Net-(D00B1-Pad2)
- D00G2 pad 2: unconnected-(D00G2-Pad2) -> Net-(D00F2-Pad2)
- D00H1 pad 2: unconnected-(D00H1-Pad2) -> Net-(D00B1-Pad2)
- D00H2 pad 2: unconnected-(D00H2-Pad2) -> Net-(D00F2-Pad2)
- D01A1 pad 2: unconnected-(D01A1-Pad2) -> Net-(D01B1-Pad2)
- D01A2 pad 2: unconnected-(D01A2-Pad2) -> Net-(D01E2-Pad2)
- D01B1 pad 2: unconnected-(D01B1-Pad2) -> Net-(D01B1-Pad2)
- D01B2 pad 2: unconnected-(D01B2-Pad2) -> Net-(D01E2-Pad2)
- D01C1 pad 2: unconnected-(D01C1-Pad2) -> Net-(D01B1-Pad2)
- D01C2 pad 2: unconnected-(D01C2-Pad2) -> Net-(D01E2-Pad2)
- D01D1 pad 2: unconnected-(D01D1-Pad2) -> Net-(D01B1-Pad2)
- D01D2 pad 2: unconnected-(D01D2-Pad2) -> Net-(D01E2-Pad2)
- D01E1 pad 2: unconnected-(D01E1-Pad2) -> Net-(D01B1-Pad2)
- D01E2 pad 2: unconnected-(D01E2-Pad2) -> Net-(D01E2-Pad2)
- D01F1 pad 2: unconnected-(D01F1-Pad2) -> Net-(D01B1-Pad2)
- D01F2 pad 2: unconnected-(D01F2-Pad2) -> Net-(D01E2-Pad2)
- D01G1 pad 2: unconnected-(D01G1-Pad2) -> Net-(D01B1-Pad2)
- D01G2 pad 2: unconnected-(D01G2-Pad2) -> Net-(D01E2-Pad2)
- D01H1 pad 2: unconnected-(D01H1-Pad2) -> Net-(D01B1-Pad2)
- D01H2 pad 2: unconnected-(D01H2-Pad2) -> Net-(D01E2-Pad2)
- D02A1 pad 2: unconnected-(D02A1-Pad2) -> Net-(D02B1-Pad2)
- D02A2 pad 2: unconnected-(D02A2-Pad2) -> Net-(D02G2-Pad2)
- D02B1 pad 2: unconnected-(D02B1-Pad2) -> Net-(D02B1-Pad2)
- D02B2 pad 2: unconnected-(D02B2-Pad2) -> Net-(D02G2-Pad2)
- D02C1 pad 2: unconnected-(D02C1-Pad2) -> Net-(D02B1-Pad2)
- D02C2 pad 2: unconnected-(D02C2-Pad2) -> Net-(D02G2-Pad2)
- D02D1 pad 2: unconnected-(D02D1-Pad2) -> Net-(D02B1-Pad2)
- D02D2 pad 2: unconnected-(D02D2-Pad2) -> Net-(D02G2-Pad2)
- D02E1 pad 2: unconnected-(D02E1-Pad2) -> Net-(D02B1-Pad2)
- D02E2 pad 2: unconnected-(D02E2-Pad2) -> Net-(D02G2-Pad2)
- D02F1 pad 2: unconnected-(D02F1-Pad2) -> Net-(D02B1-Pad2)
- D02F2 pad 2: unconnected-(D02F2-Pad2) -> Net-(D02G2-Pad2)
- D02G1 pad 2: unconnected-(D02G1-Pad2) -> Net-(D02B1-Pad2)
- D02G2 pad 2: unconnected-(D02G2-Pad2) -> Net-(D02G2-Pad2)
- D02H1 pad 2: unconnected-(D02H1-Pad2) -> Net-(D02B1-Pad2)
- D02H2 pad 2: unconnected-(D02H2-Pad2) -> Net-(D02G2-Pad2)
- D03A1 pad 2: unconnected-(D03A1-Pad2) -> Net-(D03A1-Pad2)
- D03A2 pad 2: unconnected-(D03A2-Pad2) -> Net-(D03G2-Pad2)
- D03B1 pad 2: unconnected-(D03B1-Pad2) -> Net-(D03A1-Pad2)
- D03B2 pad 2: unconnected-(D03B2-Pad2) -> Net-(D03G2-Pad2)
- D03C1 pad 2: unconnected-(D03C1-Pad2) -> Net-(D03A1-Pad2)
- D03C2 pad 2: unconnected-(D03C2-Pad2) -> Net-(D03G2-Pad2)
- D03D1 pad 2: unconnected-(D03D1-Pad2) -> Net-(D03A1-Pad2)
- D03D2 pad 2: unconnected-(D03D2-Pad2) -> Net-(D03G2-Pad2)
- D03E1 pad 2: unconnected-(D03E1-Pad2) -> Net-(D03A1-Pad2)
- D03E2 pad 2: unconnected-(D03E2-Pad2) -> Net-(D03G2-Pad2)
- D03F1 pad 2: unconnected-(D03F1-Pad2) -> Net-(D03A1-Pad2)
- D03F2 pad 2: unconnected-(D03F2-Pad2) -> Net-(D03G2-Pad2)
- D03G1 pad 2: unconnected-(D03G1-Pad2) -> Net-(D03A1-Pad2)
- D03G2 pad 2: unconnected-(D03G2-Pad2) -> Net-(D03G2-Pad2)
- D03H1 pad 2: unconnected-(D03H1-Pad2) -> Net-(D03A1-Pad2)
- D03H2 pad 2: unconnected-(D03H2-Pad2) -> Net-(D03G2-Pad2)
- D04A1 pad 2: unconnected-(D04A1-Pad2) -> Net-(D04E1-Pad2)
- D04A2 pad 2: unconnected-(D04A2-Pad2) -> Net-(R37-Pad2)
- D04B1 pad 2: unconnected-(D04B1-Pad2) -> Net-(D04E1-Pad2)
- D04B2 pad 2: unconnected-(D04B2-Pad2) -> Net-(R37-Pad2)
- D04C1 pad 2: unconnected-(D04C1-Pad2) -> Net-(D04E1-Pad2)
- D04C2 pad 2: unconnected-(D04C2-Pad2) -> Net-(R37-Pad2)
- D04D1 pad 2: unconnected-(D04D1-Pad2) -> Net-(D04E1-Pad2)
- D04D2 pad 2: unconnected-(D04D2-Pad2) -> Net-(R37-Pad2)
- D04E1 pad 2: unconnected-(D04E1-Pad2) -> Net-(D04E1-Pad2)
- D04E2 pad 2: unconnected-(D04E2-Pad2) -> Net-(R37-Pad2)
- D04F1 pad 2: unconnected-(D04F1-Pad2) -> Net-(D04E1-Pad2)
- D04F2 pad 2: unconnected-(D04F2-Pad2) -> Net-(R37-Pad2)
- D04G1 pad 2: unconnected-(D04G1-Pad2) -> Net-(D04E1-Pad2)
- D04G2 pad 2: unconnected-(D04G2-Pad2) -> Net-(R37-Pad2)
- D04H1 pad 2: unconnected-(D04H1-Pad2) -> Net-(D04E1-Pad2)
- D04H2 pad 2: unconnected-(D04H2-Pad2) -> Net-(R37-Pad2)
- D05A1 pad 2: unconnected-(D05A1-Pad2) -> Net-(D05E1-Pad2)
- D05A2 pad 2: unconnected-(D05A2-Pad2) -> Net-(R38-Pad2)
- D05B1 pad 2: unconnected-(D05B1-Pad2) -> Net-(D05E1-Pad2)
- D05B2 pad 2: unconnected-(D05B2-Pad2) -> Net-(R38-Pad2)
- D05C1 pad 2: unconnected-(D05C1-Pad2) -> Net-(D05E1-Pad2)
- D05C2 pad 2: unconnected-(D05C2-Pad2) -> Net-(R38-Pad2)
- D05D1 pad 2: unconnected-(D05D1-Pad2) -> Net-(D05E1-Pad2)
- D05D2 pad 2: unconnected-(D05D2-Pad2) -> Net-(R38-Pad2)
- D05E1 pad 2: unconnected-(D05E1-Pad2) -> Net-(D05E1-Pad2)
- D05E2 pad 2: unconnected-(D05E2-Pad2) -> Net-(R38-Pad2)
- D05F1 pad 2: unconnected-(D05F1-Pad2) -> Net-(D05E1-Pad2)
- D05F2 pad 2: unconnected-(D05F2-Pad2) -> Net-(R38-Pad2)
- D05G1 pad 2: unconnected-(D05G1-Pad2) -> Net-(D05E1-Pad2)
- D05G2 pad 2: unconnected-(D05G2-Pad2) -> Net-(R38-Pad2)
- D05H1 pad 2: unconnected-(D05H1-Pad2) -> Net-(D05E1-Pad2)
- D05H2 pad 2: unconnected-(D05H2-Pad2) -> Net-(R38-Pad2)
- D06A1 pad 2: unconnected-(D06A1-Pad2) -> Net-(D06H1-Pad2)
- D06A2 pad 2: unconnected-(D06A2-Pad2) -> Net-(R39-Pad2)
- D06B1 pad 2: unconnected-(D06B1-Pad2) -> Net-(D06H1-Pad2)
- D06B2 pad 2: unconnected-(D06B2-Pad2) -> Net-(R39-Pad2)
- D06C1 pad 2: unconnected-(D06C1-Pad2) -> Net-(D06H1-Pad2)
- D06C2 pad 2: unconnected-(D06C2-Pad2) -> Net-(R39-Pad2)
- D06D1 pad 2: unconnected-(D06D1-Pad2) -> Net-(D06H1-Pad2)
- D06D2 pad 2: unconnected-(D06D2-Pad2) -> Net-(R39-Pad2)
- D06E1 pad 2: unconnected-(D06E1-Pad2) -> Net-(D06H1-Pad2)
- D06E2 pad 2: unconnected-(D06E2-Pad2) -> Net-(R39-Pad2)
- D06F1 pad 2: unconnected-(D06F1-Pad2) -> Net-(D06H1-Pad2)
- D06F2 pad 2: unconnected-(D06F2-Pad2) -> Net-(R39-Pad2)
- D06G1 pad 2: unconnected-(D06G1-Pad2) -> Net-(D06H1-Pad2)
- D06G2 pad 2: unconnected-(D06G2-Pad2) -> Net-(R39-Pad2)
- D06H1 pad 2: unconnected-(D06H1-Pad2) -> Net-(D06H1-Pad2)
- D06H2 pad 2: unconnected-(D06H2-Pad2) -> Net-(R39-Pad2)
- D07A1 pad 2: unconnected-(D07A1-Pad2) -> Net-(D07H1-Pad2)
- D07A2 pad 2: unconnected-(D07A2-Pad2) -> Net-(R40-Pad2)
- D07B1 pad 2: unconnected-(D07B1-Pad2) -> Net-(D07H1-Pad2)
- D07B2 pad 2: unconnected-(D07B2-Pad2) -> Net-(R40-Pad2)
- D07C1 pad 2: unconnected-(D07C1-Pad2) -> Net-(D07H1-Pad2)
- D07C2 pad 2: unconnected-(D07C2-Pad2) -> Net-(R40-Pad2)
- D07D1 pad 2: unconnected-(D07D1-Pad2) -> Net-(D07H1-Pad2)
- D07D2 pad 2: unconnected-(D07D2-Pad2) -> Net-(R40-Pad2)
- D07E1 pad 2: unconnected-(D07E1-Pad2) -> Net-(D07H1-Pad2)
- D07E2 pad 2: unconnected-(D07E2-Pad2) -> Net-(R40-Pad2)
- D07F1 pad 2: unconnected-(D07F1-Pad2) -> Net-(D07H1-Pad2)
- D07F2 pad 2: unconnected-(D07F2-Pad2) -> Net-(R40-Pad2)
- D07G1 pad 2: unconnected-(D07G1-Pad2) -> Net-(D07H1-Pad2)
- D07G2 pad 2: unconnected-(D07G2-Pad2) -> Net-(R40-Pad2)
- D07H1 pad 2: unconnected-(D07H1-Pad2) -> Net-(D07H1-Pad2)
- D07H2 pad 2: unconnected-(D07H2-Pad2) -> Net-(R40-Pad2)
- D08A1 pad 2: unconnected-(D08A1-Pad2) -> Net-(D08F1-Pad2)
- D08A2 pad 2: unconnected-(D08A2-Pad2) -> Net-(D08H2-Pad2)
- D08B1 pad 2: unconnected-(D08B1-Pad2) -> Net-(D08F1-Pad2)
- D08B2 pad 2: unconnected-(D08B2-Pad2) -> Net-(D08H2-Pad2)
- D08C1 pad 2: unconnected-(D08C1-Pad2) -> Net-(D08F1-Pad2)
- D08C2 pad 2: unconnected-(D08C2-Pad2) -> Net-(D08H2-Pad2)
- D08D1 pad 2: unconnected-(D08D1-Pad2) -> Net-(D08F1-Pad2)
- D08D2 pad 2: unconnected-(D08D2-Pad2) -> Net-(D08H2-Pad2)
- D08E1 pad 2: unconnected-(D08E1-Pad2) -> Net-(D08F1-Pad2)
- D08E2 pad 2: unconnected-(D08E2-Pad2) -> Net-(D08H2-Pad2)
- D08F1 pad 2: unconnected-(D08F1-Pad2) -> Net-(D08F1-Pad2)
- D08F2 pad 2: unconnected-(D08F2-Pad2) -> Net-(D08H2-Pad2)
- D08G1 pad 2: unconnected-(D08G1-Pad2) -> Net-(D08F1-Pad2)
- D08G2 pad 2: unconnected-(D08G2-Pad2) -> Net-(D08H2-Pad2)
- D08H1 pad 2: unconnected-(D08H1-Pad2) -> Net-(D08F1-Pad2)
- D08H2 pad 2: unconnected-(D08H2-Pad2) -> Net-(D08H2-Pad2)
- D09A1 pad 2: unconnected-(D09A1-Pad2) -> Net-(D09G1-Pad2)
- D09A2 pad 2: unconnected-(D09A2-Pad2) -> Net-(D09C2-Pad2)
- D09B1 pad 2: unconnected-(D09B1-Pad2) -> Net-(D09G1-Pad2)
- D09B2 pad 2: unconnected-(D09B2-Pad2) -> Net-(D09C2-Pad2)
- D09C1 pad 2: unconnected-(D09C1-Pad2) -> Net-(D09G1-Pad2)
- D09C2 pad 2: unconnected-(D09C2-Pad2) -> Net-(D09C2-Pad2)
- D09D1 pad 2: unconnected-(D09D1-Pad2) -> Net-(D09G1-Pad2)
- D09D2 pad 2: unconnected-(D09D2-Pad2) -> Net-(D09C2-Pad2)
- D09E1 pad 2: unconnected-(D09E1-Pad2) -> Net-(D09G1-Pad2)
- D09E2 pad 2: unconnected-(D09E2-Pad2) -> Net-(D09C2-Pad2)
- D09F1 pad 2: unconnected-(D09F1-Pad2) -> Net-(D09G1-Pad2)
- D09F2 pad 2: unconnected-(D09F2-Pad2) -> Net-(D09C2-Pad2)
- D09G1 pad 2: unconnected-(D09G1-Pad2) -> Net-(D09G1-Pad2)
- D09G2 pad 2: unconnected-(D09G2-Pad2) -> Net-(D09C2-Pad2)
- D09H1 pad 2: unconnected-(D09H1-Pad2) -> Net-(D09G1-Pad2)
- D09H2 pad 2: unconnected-(D09H2-Pad2) -> Net-(D09C2-Pad2)
- D10A1 pad 2: unconnected-(D10A1-Pad2) -> Net-(D10G1-Pad2)
- D10A2 pad 2: unconnected-(D10A2-Pad2) -> Net-(D10C2-Pad2)
- D10B1 pad 2: unconnected-(D10B1-Pad2) -> Net-(D10G1-Pad2)
- D10B2 pad 2: unconnected-(D10B2-Pad2) -> Net-(D10C2-Pad2)
- D10C1 pad 2: unconnected-(D10C1-Pad2) -> Net-(D10G1-Pad2)
- D10C2 pad 2: unconnected-(D10C2-Pad2) -> Net-(D10C2-Pad2)
- D10D1 pad 2: unconnected-(D10D1-Pad2) -> Net-(D10G1-Pad2)
- D10D2 pad 2: unconnected-(D10D2-Pad2) -> Net-(D10C2-Pad2)
- D10E1 pad 2: unconnected-(D10E1-Pad2) -> Net-(D10G1-Pad2)
- D10E2 pad 2: unconnected-(D10E2-Pad2) -> Net-(D10C2-Pad2)
- D10F1 pad 2: unconnected-(D10F1-Pad2) -> Net-(D10G1-Pad2)
- D10F2 pad 2: unconnected-(D10F2-Pad2) -> Net-(D10C2-Pad2)
- D10G1 pad 2: unconnected-(D10G1-Pad2) -> Net-(D10G1-Pad2)
- D10G2 pad 2: unconnected-(D10G2-Pad2) -> Net-(D10C2-Pad2)
- D10H1 pad 2: unconnected-(D10H1-Pad2) -> Net-(D10G1-Pad2)
- D10H2 pad 2: unconnected-(D10H2-Pad2) -> Net-(D10C2-Pad2)
- D11A1 pad 2: unconnected-(D11A1-Pad2) -> Net-(D11F1-Pad2)
- D11A2 pad 2: unconnected-(D11A2-Pad2) -> Net-(D11C2-Pad2)
- D11B1 pad 2: unconnected-(D11B1-Pad2) -> Net-(D11F1-Pad2)
- D11B2 pad 2: unconnected-(D11B2-Pad2) -> Net-(D11C2-Pad2)
- D11C1 pad 2: unconnected-(D11C1-Pad2) -> Net-(D11F1-Pad2)
- D11C2 pad 2: unconnected-(D11C2-Pad2) -> Net-(D11C2-Pad2)
- D11D1 pad 2: unconnected-(D11D1-Pad2) -> Net-(D11F1-Pad2)
- D11D2 pad 2: unconnected-(D11D2-Pad2) -> Net-(D11C2-Pad2)
- D11E1 pad 2: unconnected-(D11E1-Pad2) -> Net-(D11F1-Pad2)
- D11E2 pad 2: unconnected-(D11E2-Pad2) -> Net-(D11C2-Pad2)
- D11F1 pad 2: unconnected-(D11F1-Pad2) -> Net-(D11F1-Pad2)
- D11F2 pad 2: unconnected-(D11F2-Pad2) -> Net-(D11C2-Pad2)
- D11G1 pad 2: unconnected-(D11G1-Pad2) -> Net-(D11F1-Pad2)
- D11G2 pad 2: unconnected-(D11G2-Pad2) -> Net-(D11C2-Pad2)
- D11H1 pad 2: unconnected-(D11H1-Pad2) -> Net-(D11F1-Pad2)
- D11H2 pad 2: unconnected-(D11H2-Pad2) -> Net-(D11C2-Pad2)
- D12A1 pad 2: unconnected-(D12A1-Pad2) -> Net-(D12F1-Pad2)
- D12A2 pad 2: unconnected-(D12A2-Pad2) -> Net-(D12G2-Pad2)
- D12B1 pad 2: unconnected-(D12B1-Pad2) -> Net-(D12F1-Pad2)
- D12B2 pad 2: unconnected-(D12B2-Pad2) -> Net-(D12G2-Pad2)
- D12C1 pad 2: unconnected-(D12C1-Pad2) -> Net-(D12F1-Pad2)
- D12C2 pad 2: unconnected-(D12C2-Pad2) -> Net-(D12G2-Pad2)
- D12D1 pad 2: unconnected-(D12D1-Pad2) -> Net-(D12F1-Pad2)
- D12D2 pad 2: unconnected-(D12D2-Pad2) -> Net-(D12G2-Pad2)
- D12E1 pad 2: unconnected-(D12E1-Pad2) -> Net-(D12F1-Pad2)
- D12E2 pad 2: unconnected-(D12E2-Pad2) -> Net-(D12G2-Pad2)
- D12F1 pad 2: unconnected-(D12F1-Pad2) -> Net-(D12F1-Pad2)
- D12F2 pad 2: unconnected-(D12F2-Pad2) -> Net-(D12G2-Pad2)
- D12G1 pad 2: unconnected-(D12G1-Pad2) -> Net-(D12F1-Pad2)
- D12G2 pad 2: unconnected-(D12G2-Pad2) -> Net-(D12G2-Pad2)
- D12H1 pad 2: unconnected-(D12H1-Pad2) -> Net-(D12F1-Pad2)
- D12H2 pad 2: unconnected-(D12H2-Pad2) -> Net-(D12G2-Pad2)
- D13A1 pad 2: unconnected-(D13A1-Pad2) -> Net-(D13F1-Pad2)
- D13A2 pad 2: unconnected-(D13A2-Pad2) -> Net-(R46-Pad2)
- D13B1 pad 2: unconnected-(D13B1-Pad2) -> Net-(D13F1-Pad2)
- D13B2 pad 2: unconnected-(D13B2-Pad2) -> Net-(R46-Pad2)
- D13C1 pad 2: unconnected-(D13C1-Pad2) -> Net-(D13F1-Pad2)
- D13C2 pad 2: unconnected-(D13C2-Pad2) -> Net-(R46-Pad2)
- D13D1 pad 2: unconnected-(D13D1-Pad2) -> Net-(D13F1-Pad2)
- D13D2 pad 2: unconnected-(D13D2-Pad2) -> Net-(R46-Pad2)
- D13E1 pad 2: unconnected-(D13E1-Pad2) -> Net-(D13F1-Pad2)
- D13E2 pad 2: unconnected-(D13E2-Pad2) -> Net-(R46-Pad2)
- D13F1 pad 2: unconnected-(D13F1-Pad2) -> Net-(D13F1-Pad2)
- D13F2 pad 2: unconnected-(D13F2-Pad2) -> Net-(R46-Pad2)
- D13G1 pad 2: unconnected-(D13G1-Pad2) -> Net-(D13F1-Pad2)
- D13G2 pad 2: unconnected-(D13G2-Pad2) -> Net-(R46-Pad2)
- D13H1 pad 2: unconnected-(D13H1-Pad2) -> Net-(D13F1-Pad2)
- D13H2 pad 2: unconnected-(D13H2-Pad2) -> Net-(R46-Pad2)
- D14A1 pad 2: unconnected-(D14A1-Pad2) -> Net-(D14A1-Pad2)
- D14A2 pad 2: unconnected-(D14A2-Pad2) -> Net-(D14F2-Pad2)
- D14B1 pad 2: unconnected-(D14B1-Pad2) -> Net-(D14A1-Pad2)
- D14B2 pad 2: unconnected-(D14B2-Pad2) -> Net-(D14F2-Pad2)
- D14C1 pad 2: unconnected-(D14C1-Pad2) -> Net-(D14A1-Pad2)
- D14C2 pad 2: unconnected-(D14C2-Pad2) -> Net-(D14F2-Pad2)
- D14D1 pad 2: unconnected-(D14D1-Pad2) -> Net-(D14A1-Pad2)
- D14D2 pad 2: unconnected-(D14D2-Pad2) -> Net-(D14F2-Pad2)
- D14E1 pad 2: unconnected-(D14E1-Pad2) -> Net-(D14A1-Pad2)
- D14E2 pad 2: unconnected-(D14E2-Pad2) -> Net-(D14F2-Pad2)
- D14F1 pad 2: unconnected-(D14F1-Pad2) -> Net-(D14A1-Pad2)
- D14F2 pad 2: unconnected-(D14F2-Pad2) -> Net-(D14F2-Pad2)
- D14G1 pad 2: unconnected-(D14G1-Pad2) -> Net-(D14A1-Pad2)
- D14G2 pad 2: unconnected-(D14G2-Pad2) -> Net-(D14F2-Pad2)
- D14H1 pad 2: unconnected-(D14H1-Pad2) -> Net-(D14A1-Pad2)
- D14H2 pad 2: unconnected-(D14H2-Pad2) -> Net-(D14F2-Pad2)
- D15A1 pad 2: unconnected-(D15A1-Pad2) -> Net-(D15H1-Pad2)
- D15A2 pad 2: unconnected-(D15A2-Pad2) -> Net-(D15F2-Pad2)
- D15B1 pad 2: unconnected-(D15B1-Pad2) -> Net-(D15H1-Pad2)
- D15B2 pad 2: unconnected-(D15B2-Pad2) -> Net-(D15F2-Pad2)
- D15C1 pad 2: unconnected-(D15C1-Pad2) -> Net-(D15H1-Pad2)
- D15C2 pad 2: unconnected-(D15C2-Pad2) -> Net-(D15F2-Pad2)
- D15D1 pad 2: unconnected-(D15D1-Pad2) -> Net-(D15H1-Pad2)
- D15D2 pad 2: unconnected-(D15D2-Pad2) -> Net-(D15F2-Pad2)
- D15E1 pad 2: unconnected-(D15E1-Pad2) -> Net-(D15H1-Pad2)
- D15E2 pad 2: unconnected-(D15E2-Pad2) -> Net-(D15F2-Pad2)
- D15F1 pad 2: unconnected-(D15F1-Pad2) -> Net-(D15H1-Pad2)
- D15F2 pad 2: unconnected-(D15F2-Pad2) -> Net-(D15F2-Pad2)
- D15G1 pad 2: unconnected-(D15G1-Pad2) -> Net-(D15H1-Pad2)
- D15G2 pad 2: unconnected-(D15G2-Pad2) -> Net-(D15F2-Pad2)
- D15H1 pad 2: unconnected-(D15H1-Pad2) -> Net-(D15H1-Pad2)
- D15H2 pad 2: unconnected-(D15H2-Pad2) -> Net-(D15F2-Pad2)
- D16A1 pad 2: unconnected-(D16A1-Pad2) -> Net-(D16G1-Pad2)
- D16A2 pad 2: unconnected-(D16A2-Pad2) -> Net-(D16H2-Pad2)
- D16B1 pad 2: unconnected-(D16B1-Pad2) -> Net-(D16G1-Pad2)
- D16B2 pad 2: unconnected-(D16B2-Pad2) -> Net-(D16H2-Pad2)
- D16C1 pad 2: unconnected-(D16C1-Pad2) -> Net-(D16G1-Pad2)
- D16C2 pad 2: unconnected-(D16C2-Pad2) -> Net-(D16H2-Pad2)
- D16D1 pad 2: unconnected-(D16D1-Pad2) -> Net-(D16G1-Pad2)
- D16D2 pad 2: unconnected-(D16D2-Pad2) -> Net-(D16H2-Pad2)
- D16E1 pad 2: unconnected-(D16E1-Pad2) -> Net-(D16G1-Pad2)
- D16E2 pad 2: unconnected-(D16E2-Pad2) -> Net-(D16H2-Pad2)
- D16F1 pad 2: unconnected-(D16F1-Pad2) -> Net-(D16G1-Pad2)
- D16F2 pad 2: unconnected-(D16F2-Pad2) -> Net-(D16H2-Pad2)
- D16G1 pad 2: unconnected-(D16G1-Pad2) -> Net-(D16G1-Pad2)
- D16G2 pad 2: unconnected-(D16G2-Pad2) -> Net-(D16H2-Pad2)
- D16H1 pad 2: unconnected-(D16H1-Pad2) -> Net-(D16G1-Pad2)
- D16H2 pad 2: unconnected-(D16H2-Pad2) -> Net-(D16H2-Pad2)
- D17A1 pad 2: unconnected-(D17A1-Pad2) -> Net-(D17H1-Pad2)
- D17A2 pad 2: unconnected-(D17A2-Pad2) -> Net-(R50-Pad2)
- D17B1 pad 2: unconnected-(D17B1-Pad2) -> Net-(D17H1-Pad2)
- D17B2 pad 2: unconnected-(D17B2-Pad2) -> Net-(R50-Pad2)
- D17C1 pad 2: unconnected-(D17C1-Pad2) -> Net-(D17H1-Pad2)
- D17C2 pad 2: unconnected-(D17C2-Pad2) -> Net-(R50-Pad2)
- D17D1 pad 2: unconnected-(D17D1-Pad2) -> Net-(D17H1-Pad2)
- D17D2 pad 2: unconnected-(D17D2-Pad2) -> Net-(R50-Pad2)
- D17E1 pad 2: unconnected-(D17E1-Pad2) -> Net-(D17H1-Pad2)
- D17E2 pad 2: unconnected-(D17E2-Pad2) -> Net-(R50-Pad2)
- D17F1 pad 2: unconnected-(D17F1-Pad2) -> Net-(D17H1-Pad2)
- D17F2 pad 2: unconnected-(D17F2-Pad2) -> Net-(R50-Pad2)
- D17G1 pad 2: unconnected-(D17G1-Pad2) -> Net-(D17H1-Pad2)
- D17G2 pad 2: unconnected-(D17G2-Pad2) -> Net-(R50-Pad2)
- D17H1 pad 2: unconnected-(D17H1-Pad2) -> Net-(D17H1-Pad2)
- D17H2 pad 2: unconnected-(D17H2-Pad2) -> Net-(R50-Pad2)
- D18A1 pad 2: unconnected-(D18A1-Pad2) -> Net-(D18E1-Pad2)
- D18A2 pad 2: unconnected-(D18A2-Pad2) -> Net-(D18H2-Pad2)
- D18B1 pad 2: unconnected-(D18B1-Pad2) -> Net-(D18E1-Pad2)
- D18B2 pad 2: unconnected-(D18B2-Pad2) -> Net-(D18H2-Pad2)
- D18C1 pad 2: unconnected-(D18C1-Pad2) -> Net-(D18E1-Pad2)
- D18C2 pad 2: unconnected-(D18C2-Pad2) -> Net-(D18H2-Pad2)
- D18D1 pad 2: unconnected-(D18D1-Pad2) -> Net-(D18E1-Pad2)
- D18D2 pad 2: unconnected-(D18D2-Pad2) -> Net-(D18H2-Pad2)
- D18E1 pad 2: unconnected-(D18E1-Pad2) -> Net-(D18E1-Pad2)
- D18E2 pad 2: unconnected-(D18E2-Pad2) -> Net-(D18H2-Pad2)
- D18F1 pad 2: unconnected-(D18F1-Pad2) -> Net-(D18E1-Pad2)
- D18F2 pad 2: unconnected-(D18F2-Pad2) -> Net-(D18H2-Pad2)
- D18G1 pad 2: unconnected-(D18G1-Pad2) -> Net-(D18E1-Pad2)
- D18G2 pad 2: unconnected-(D18G2-Pad2) -> Net-(D18H2-Pad2)
- D18H1 pad 2: unconnected-(D18H1-Pad2) -> Net-(D18E1-Pad2)
- D18H2 pad 2: unconnected-(D18H2-Pad2) -> Net-(D18H2-Pad2)
- D19A1 pad 2: unconnected-(D19A1-Pad2) -> Net-(D19H1-Pad2)
- D19A2 pad 2: unconnected-(D19A2-Pad2) -> Net-(D19H2-Pad2)
- D19B1 pad 2: unconnected-(D19B1-Pad2) -> Net-(D19H1-Pad2)
- D19B2 pad 2: unconnected-(D19B2-Pad2) -> Net-(D19H2-Pad2)
- D19C1 pad 2: unconnected-(D19C1-Pad2) -> Net-(D19H1-Pad2)
- D19C2 pad 2: unconnected-(D19C2-Pad2) -> Net-(D19H2-Pad2)
- D19D1 pad 2: unconnected-(D19D1-Pad2) -> Net-(D19H1-Pad2)
- D19D2 pad 2: unconnected-(D19D2-Pad2) -> Net-(D19H2-Pad2)
- D19E1 pad 2: unconnected-(D19E1-Pad2) -> Net-(D19H1-Pad2)
- D19E2 pad 2: unconnected-(D19E2-Pad2) -> Net-(D19H2-Pad2)
- D19F1 pad 2: unconnected-(D19F1-Pad2) -> Net-(D19H1-Pad2)
- D19F2 pad 2: unconnected-(D19F2-Pad2) -> Net-(D19H2-Pad2)
- D19G1 pad 2: unconnected-(D19G1-Pad2) -> Net-(D19H1-Pad2)
- D19G2 pad 2: unconnected-(D19G2-Pad2) -> Net-(D19H2-Pad2)
- D19H1 pad 2: unconnected-(D19H1-Pad2) -> Net-(D19H1-Pad2)
- D19H2 pad 2: unconnected-(D19H2-Pad2) -> Net-(D19H2-Pad2)
- D20A1 pad 2: unconnected-(D20A1-Pad2) -> Net-(D20H1-Pad2)
- D20A2 pad 2: unconnected-(D20A2-Pad2) -> Net-(D20A2-Pad2)
- D20B1 pad 2: unconnected-(D20B1-Pad2) -> Net-(D20H1-Pad2)
- D20B2 pad 2: unconnected-(D20B2-Pad2) -> Net-(D20A2-Pad2)
- D20C1 pad 2: unconnected-(D20C1-Pad2) -> Net-(D20H1-Pad2)
- D20C2 pad 2: unconnected-(D20C2-Pad2) -> Net-(D20A2-Pad2)
- D20D1 pad 2: unconnected-(D20D1-Pad2) -> Net-(D20H1-Pad2)
- D20D2 pad 2: unconnected-(D20D2-Pad2) -> Net-(D20A2-Pad2)
- D20E1 pad 2: unconnected-(D20E1-Pad2) -> Net-(D20H1-Pad2)
- D20E2 pad 2: unconnected-(D20E2-Pad2) -> Net-(D20A2-Pad2)
- D20F1 pad 2: unconnected-(D20F1-Pad2) -> Net-(D20H1-Pad2)
- D20F2 pad 2: unconnected-(D20F2-Pad2) -> Net-(D20A2-Pad2)
- D20G1 pad 2: unconnected-(D20G1-Pad2) -> Net-(D20H1-Pad2)
- D20G2 pad 2: unconnected-(D20G2-Pad2) -> Net-(D20A2-Pad2)
- D20H1 pad 2: unconnected-(D20H1-Pad2) -> Net-(D20H1-Pad2)
- D20H2 pad 2: unconnected-(D20H2-Pad2) -> Net-(D20A2-Pad2)
- D21A1 pad 2: unconnected-(D21A1-Pad2) -> Net-(R22-Pad2)
- D21A2 pad 2: unconnected-(D21A2-Pad2) -> Net-(D21B2-Pad2)
- D21B1 pad 2: unconnected-(D21B1-Pad2) -> Net-(R22-Pad2)
- D21B2 pad 2: unconnected-(D21B2-Pad2) -> Net-(D21B2-Pad2)
- D21C1 pad 2: unconnected-(D21C1-Pad2) -> Net-(R22-Pad2)
- D21C2 pad 2: unconnected-(D21C2-Pad2) -> Net-(D21B2-Pad2)
- D21D1 pad 2: unconnected-(D21D1-Pad2) -> Net-(R22-Pad2)
- D21D2 pad 2: unconnected-(D21D2-Pad2) -> Net-(D21B2-Pad2)
- D21E1 pad 2: unconnected-(D21E1-Pad2) -> Net-(R22-Pad2)
- D21E2 pad 2: unconnected-(D21E2-Pad2) -> Net-(D21B2-Pad2)
- D21F1 pad 2: unconnected-(D21F1-Pad2) -> Net-(R22-Pad2)
- D21F2 pad 2: unconnected-(D21F2-Pad2) -> Net-(D21B2-Pad2)
- D21G1 pad 2: unconnected-(D21G1-Pad2) -> Net-(R22-Pad2)
- D21G2 pad 2: unconnected-(D21G2-Pad2) -> Net-(D21B2-Pad2)
- D21H1 pad 2: unconnected-(D21H1-Pad2) -> Net-(R22-Pad2)
- D21H2 pad 2: unconnected-(D21H2-Pad2) -> Net-(D21B2-Pad2)
- D22A1 pad 2: unconnected-(D22A1-Pad2) -> Net-(D22F1-Pad2)
- D22A2 pad 2: unconnected-(D22A2-Pad2) -> Net-(D22G2-Pad2)
- D22B1 pad 2: unconnected-(D22B1-Pad2) -> Net-(D22F1-Pad2)
- D22B2 pad 2: unconnected-(D22B2-Pad2) -> Net-(D22G2-Pad2)
- D22C1 pad 2: unconnected-(D22C1-Pad2) -> Net-(D22F1-Pad2)
- D22C2 pad 2: unconnected-(D22C2-Pad2) -> Net-(D22G2-Pad2)
- D22D1 pad 2: unconnected-(D22D1-Pad2) -> Net-(D22F1-Pad2)
- D22D2 pad 2: unconnected-(D22D2-Pad2) -> Net-(D22G2-Pad2)
- D22E1 pad 2: unconnected-(D22E1-Pad2) -> Net-(D22F1-Pad2)
- D22E2 pad 2: unconnected-(D22E2-Pad2) -> Net-(D22G2-Pad2)
- D22F1 pad 2: unconnected-(D22F1-Pad2) -> Net-(D22F1-Pad2)
- D22F2 pad 2: unconnected-(D22F2-Pad2) -> Net-(D22G2-Pad2)
- D22G1 pad 2: unconnected-(D22G1-Pad2) -> Net-(D22F1-Pad2)
- D22G2 pad 2: unconnected-(D22G2-Pad2) -> Net-(D22G2-Pad2)
- D22H1 pad 2: unconnected-(D22H1-Pad2) -> Net-(D22F1-Pad2)
- D22H2 pad 2: unconnected-(D22H2-Pad2) -> Net-(D22G2-Pad2)
- D23A1 pad 2: unconnected-(D23A1-Pad2) -> Net-(R24-Pad2)
- D23A2 pad 2: unconnected-(D23A2-Pad2) -> Net-(D23A2-Pad2)
- D23B1 pad 2: unconnected-(D23B1-Pad2) -> Net-(R24-Pad2)
- D23B2 pad 2: unconnected-(D23B2-Pad2) -> Net-(D23A2-Pad2)
- D23C1 pad 2: unconnected-(D23C1-Pad2) -> Net-(R24-Pad2)
- D23C2 pad 2: unconnected-(D23C2-Pad2) -> Net-(D23A2-Pad2)
- D23D1 pad 2: unconnected-(D23D1-Pad2) -> Net-(R24-Pad2)
- D23D2 pad 2: unconnected-(D23D2-Pad2) -> Net-(D23A2-Pad2)
- D23E1 pad 2: unconnected-(D23E1-Pad2) -> Net-(R24-Pad2)
- D23E2 pad 2: unconnected-(D23E2-Pad2) -> Net-(D23A2-Pad2)
- D23F1 pad 2: unconnected-(D23F1-Pad2) -> Net-(R24-Pad2)
- D23F2 pad 2: unconnected-(D23F2-Pad2) -> Net-(D23A2-Pad2)
- D23G1 pad 2: unconnected-(D23G1-Pad2) -> Net-(R24-Pad2)
- D23G2 pad 2: unconnected-(D23G2-Pad2) -> Net-(D23A2-Pad2)
- D23H1 pad 2: unconnected-(D23H1-Pad2) -> Net-(R24-Pad2)
- D23H2 pad 2: unconnected-(D23H2-Pad2) -> Net-(D23A2-Pad2)
- D24A1 pad 2: unconnected-(D24A1-Pad2) -> Net-(R25-Pad2)
- D24A2 pad 2: unconnected-(D24A2-Pad2) -> Net-(R57-Pad2)
- D24B1 pad 2: unconnected-(D24B1-Pad2) -> Net-(R25-Pad2)
- D24B2 pad 2: unconnected-(D24B2-Pad2) -> Net-(R57-Pad2)
- D24C1 pad 2: unconnected-(D24C1-Pad2) -> Net-(R25-Pad2)
- D24C2 pad 2: unconnected-(D24C2-Pad2) -> Net-(R57-Pad2)
- D24D1 pad 2: unconnected-(D24D1-Pad2) -> Net-(R25-Pad2)
- D24D2 pad 2: unconnected-(D24D2-Pad2) -> Net-(R57-Pad2)
- D24E1 pad 2: unconnected-(D24E1-Pad2) -> Net-(R25-Pad2)
- D24E2 pad 2: unconnected-(D24E2-Pad2) -> Net-(R57-Pad2)
- D24F1 pad 2: unconnected-(D24F1-Pad2) -> Net-(R25-Pad2)
- D24F2 pad 2: unconnected-(D24F2-Pad2) -> Net-(R57-Pad2)
- D24G1 pad 2: unconnected-(D24G1-Pad2) -> Net-(R25-Pad2)
- D24G2 pad 2: unconnected-(D24G2-Pad2) -> Net-(R57-Pad2)
- D24H1 pad 2: unconnected-(D24H1-Pad2) -> Net-(R25-Pad2)
- D24H2 pad 2: unconnected-(D24H2-Pad2) -> Net-(R57-Pad2)
- D25A1 pad 2: unconnected-(D25A1-Pad2) -> Net-(R26-Pad2)
- D25A2 pad 2: unconnected-(D25A2-Pad2) -> Net-(D25H2-Pad2)
- D25B1 pad 2: unconnected-(D25B1-Pad2) -> Net-(R26-Pad2)
- D25B2 pad 2: unconnected-(D25B2-Pad2) -> Net-(D25H2-Pad2)
- D25C1 pad 2: unconnected-(D25C1-Pad2) -> Net-(R26-Pad2)
- D25C2 pad 2: unconnected-(D25C2-Pad2) -> Net-(D25H2-Pad2)
- D25D1 pad 2: unconnected-(D25D1-Pad2) -> Net-(R26-Pad2)
- D25D2 pad 2: unconnected-(D25D2-Pad2) -> Net-(D25H2-Pad2)
- D25E1 pad 2: unconnected-(D25E1-Pad2) -> Net-(R26-Pad2)
- D25E2 pad 2: unconnected-(D25E2-Pad2) -> Net-(D25H2-Pad2)
- D25F1 pad 2: unconnected-(D25F1-Pad2) -> Net-(R26-Pad2)
- D25F2 pad 2: unconnected-(D25F2-Pad2) -> Net-(D25H2-Pad2)
- D25G1 pad 2: unconnected-(D25G1-Pad2) -> Net-(R26-Pad2)
- D25G2 pad 2: unconnected-(D25G2-Pad2) -> Net-(D25H2-Pad2)
- D25H1 pad 2: unconnected-(D25H1-Pad2) -> Net-(R26-Pad2)
- D25H2 pad 2: unconnected-(D25H2-Pad2) -> Net-(D25H2-Pad2)
- D26A1 pad 2: unconnected-(D26A1-Pad2) -> Net-(D26A1-Pad2)
- D26A2 pad 2: unconnected-(D26A2-Pad2) -> Net-(R59-Pad2)
- D26B1 pad 2: unconnected-(D26B1-Pad2) -> Net-(D26A1-Pad2)
- D26B2 pad 2: unconnected-(D26B2-Pad2) -> Net-(R59-Pad2)
- D26C1 pad 2: unconnected-(D26C1-Pad2) -> Net-(D26A1-Pad2)
- D26C2 pad 2: unconnected-(D26C2-Pad2) -> Net-(R59-Pad2)
- D26D1 pad 2: unconnected-(D26D1-Pad2) -> Net-(D26A1-Pad2)
- D26D2 pad 2: unconnected-(D26D2-Pad2) -> Net-(R59-Pad2)
- D26E1 pad 2: unconnected-(D26E1-Pad2) -> Net-(D26A1-Pad2)
- D26E2 pad 2: unconnected-(D26E2-Pad2) -> Net-(R59-Pad2)
- D26F1 pad 2: unconnected-(D26F1-Pad2) -> Net-(D26A1-Pad2)
- D26F2 pad 2: unconnected-(D26F2-Pad2) -> Net-(R59-Pad2)
- D26G1 pad 2: unconnected-(D26G1-Pad2) -> Net-(D26A1-Pad2)
- D26G2 pad 2: unconnected-(D26G2-Pad2) -> Net-(R59-Pad2)
- D26H1 pad 2: unconnected-(D26H1-Pad2) -> Net-(D26A1-Pad2)
- D26H2 pad 2: unconnected-(D26H2-Pad2) -> Net-(R59-Pad2)
- D27A1 pad 2: unconnected-(D27A1-Pad2) -> Net-(D27A1-Pad2)
- D27A2 pad 2: unconnected-(D27A2-Pad2) -> Net-(D27H2-Pad2)
- D27B1 pad 2: unconnected-(D27B1-Pad2) -> Net-(D27A1-Pad2)
- D27B2 pad 2: unconnected-(D27B2-Pad2) -> Net-(D27H2-Pad2)
- D27C1 pad 2: unconnected-(D27C1-Pad2) -> Net-(D27A1-Pad2)
- D27C2 pad 2: unconnected-(D27C2-Pad2) -> Net-(D27H2-Pad2)
- D27D1 pad 2: unconnected-(D27D1-Pad2) -> Net-(D27A1-Pad2)
- D27D2 pad 2: unconnected-(D27D2-Pad2) -> Net-(D27H2-Pad2)
- D27E1 pad 2: unconnected-(D27E1-Pad2) -> Net-(D27A1-Pad2)
- D27E2 pad 2: unconnected-(D27E2-Pad2) -> Net-(D27H2-Pad2)
- D27F1 pad 2: unconnected-(D27F1-Pad2) -> Net-(D27A1-Pad2)
- D27F2 pad 2: unconnected-(D27F2-Pad2) -> Net-(D27H2-Pad2)
- D27G1 pad 2: unconnected-(D27G1-Pad2) -> Net-(D27A1-Pad2)
- D27G2 pad 2: unconnected-(D27G2-Pad2) -> Net-(D27H2-Pad2)
- D27H1 pad 2: unconnected-(D27H1-Pad2) -> Net-(D27A1-Pad2)
- D27H2 pad 2: unconnected-(D27H2-Pad2) -> Net-(D27H2-Pad2)
- D28A1 pad 2: unconnected-(D28A1-Pad2) -> Net-(D28A1-Pad2)
- D28A2 pad 2: unconnected-(D28A2-Pad2) -> Net-(D28H2-Pad2)
- D28B1 pad 2: unconnected-(D28B1-Pad2) -> Net-(D28A1-Pad2)
- D28B2 pad 2: unconnected-(D28B2-Pad2) -> Net-(D28H2-Pad2)
- D28C1 pad 2: unconnected-(D28C1-Pad2) -> Net-(D28A1-Pad2)
- D28C2 pad 2: unconnected-(D28C2-Pad2) -> Net-(D28H2-Pad2)
- D28D1 pad 2: unconnected-(D28D1-Pad2) -> Net-(D28A1-Pad2)
- D28D2 pad 2: unconnected-(D28D2-Pad2) -> Net-(D28H2-Pad2)
- D28E1 pad 2: unconnected-(D28E1-Pad2) -> Net-(D28A1-Pad2)
- D28E2 pad 2: unconnected-(D28E2-Pad2) -> Net-(D28H2-Pad2)
- D28F1 pad 2: unconnected-(D28F1-Pad2) -> Net-(D28A1-Pad2)
- D28F2 pad 2: unconnected-(D28F2-Pad2) -> Net-(D28H2-Pad2)
- D28G1 pad 2: unconnected-(D28G1-Pad2) -> Net-(D28A1-Pad2)
- D28G2 pad 2: unconnected-(D28G2-Pad2) -> Net-(D28H2-Pad2)
- D28H1 pad 2: unconnected-(D28H1-Pad2) -> Net-(D28A1-Pad2)
- D28H2 pad 2: unconnected-(D28H2-Pad2) -> Net-(D28H2-Pad2)
- D29A1 pad 2: unconnected-(D29A1-Pad2) -> Net-(D29B1-Pad2)
- D29A2 pad 2: unconnected-(D29A2-Pad2) -> Net-(D29H2-Pad2)
- D29B1 pad 2: unconnected-(D29B1-Pad2) -> Net-(D29B1-Pad2)
- D29B2 pad 2: unconnected-(D29B2-Pad2) -> Net-(D29H2-Pad2)
- D29C1 pad 2: unconnected-(D29C1-Pad2) -> Net-(D29B1-Pad2)
- D29C2 pad 2: unconnected-(D29C2-Pad2) -> Net-(D29H2-Pad2)
- D29D1 pad 2: unconnected-(D29D1-Pad2) -> Net-(D29B1-Pad2)
- D29D2 pad 2: unconnected-(D29D2-Pad2) -> Net-(D29H2-Pad2)
- D29E1 pad 2: unconnected-(D29E1-Pad2) -> Net-(D29B1-Pad2)
- D29E2 pad 2: unconnected-(D29E2-Pad2) -> Net-(D29H2-Pad2)
- D29F1 pad 2: unconnected-(D29F1-Pad2) -> Net-(D29B1-Pad2)
- D29F2 pad 2: unconnected-(D29F2-Pad2) -> Net-(D29H2-Pad2)
- D29G1 pad 2: unconnected-(D29G1-Pad2) -> Net-(D29B1-Pad2)
- D29G2 pad 2: unconnected-(D29G2-Pad2) -> Net-(D29H2-Pad2)
- D29H1 pad 2: unconnected-(D29H1-Pad2) -> Net-(D29B1-Pad2)
- D29H2 pad 2: unconnected-(D29H2-Pad2) -> Net-(D29H2-Pad2)
- D30A1 pad 2: unconnected-(D30A1-Pad2) -> Net-(D30A1-Pad2)
- D30A2 pad 2: unconnected-(D30A2-Pad2) -> Net-(R63-Pad2)
- D30B1 pad 2: unconnected-(D30B1-Pad2) -> Net-(D30A1-Pad2)
- D30B2 pad 2: unconnected-(D30B2-Pad2) -> Net-(R63-Pad2)
- D30C1 pad 2: unconnected-(D30C1-Pad2) -> Net-(D30A1-Pad2)
- D30C2 pad 2: unconnected-(D30C2-Pad2) -> Net-(R63-Pad2)
- D30D1 pad 2: unconnected-(D30D1-Pad2) -> Net-(D30A1-Pad2)
- D30D2 pad 2: unconnected-(D30D2-Pad2) -> Net-(R63-Pad2)
- D30E1 pad 2: unconnected-(D30E1-Pad2) -> Net-(D30A1-Pad2)
- D30E2 pad 2: unconnected-(D30E2-Pad2) -> Net-(R63-Pad2)
- D30F1 pad 2: unconnected-(D30F1-Pad2) -> Net-(D30A1-Pad2)
- D30F2 pad 2: unconnected-(D30F2-Pad2) -> Net-(R63-Pad2)
- D30G1 pad 2: unconnected-(D30G1-Pad2) -> Net-(D30A1-Pad2)
- D30G2 pad 2: unconnected-(D30G2-Pad2) -> Net-(R63-Pad2)
- D30H1 pad 2: unconnected-(D30H1-Pad2) -> Net-(D30A1-Pad2)
- D30H2 pad 2: unconnected-(D30H2-Pad2) -> Net-(R63-Pad2)
- D31A1 pad 2: unconnected-(D31A1-Pad2) -> Net-(D31B1-Pad2)
- D31A2 pad 2: unconnected-(D31A2-Pad2) -> Net-(R64-Pad2)
- D31B1 pad 2: unconnected-(D31B1-Pad2) -> Net-(D31B1-Pad2)
- D31B2 pad 2: unconnected-(D31B2-Pad2) -> Net-(R64-Pad2)
- D31C1 pad 2: unconnected-(D31C1-Pad2) -> Net-(D31B1-Pad2)
- D31C2 pad 2: unconnected-(D31C2-Pad2) -> Net-(R64-Pad2)
- D31D1 pad 2: unconnected-(D31D1-Pad2) -> Net-(D31B1-Pad2)
- D31D2 pad 2: unconnected-(D31D2-Pad2) -> Net-(R64-Pad2)
- D31E1 pad 2: unconnected-(D31E1-Pad2) -> Net-(D31B1-Pad2)
- D31E2 pad 2: unconnected-(D31E2-Pad2) -> Net-(R64-Pad2)
- D31F1 pad 2: unconnected-(D31F1-Pad2) -> Net-(D31B1-Pad2)
- D31F2 pad 2: unconnected-(D31F2-Pad2) -> Net-(R64-Pad2)
- D31G1 pad 2: unconnected-(D31G1-Pad2) -> Net-(D31B1-Pad2)
- D31G2 pad 2: unconnected-(D31G2-Pad2) -> Net-(R64-Pad2)
- D31H1 pad 2: unconnected-(D31H1-Pad2) -> Net-(D31B1-Pad2)
- D31H2 pad 2: unconnected-(D31H2-Pad2) -> Net-(R64-Pad2)
- R1 pad 2: unconnected-(R1-Pad2) -> Net-(D00B1-Pad2)
- R10 pad 2: unconnected-(R10-Pad2) -> Net-(D09G1-Pad2)
- R11 pad 2: unconnected-(R11-Pad2) -> Net-(D10G1-Pad2)
- R12 pad 2: unconnected-(R12-Pad2) -> Net-(D11F1-Pad2)
- R13 pad 2: unconnected-(R13-Pad2) -> Net-(D12F1-Pad2)
- R14 pad 2: unconnected-(R14-Pad2) -> Net-(D13F1-Pad2)
- R15 pad 2: unconnected-(R15-Pad2) -> Net-(D14A1-Pad2)
- R16 pad 2: unconnected-(R16-Pad2) -> Net-(D15H1-Pad2)
- R17 pad 2: unconnected-(R17-Pad2) -> Net-(D16G1-Pad2)
- R18 pad 2: unconnected-(R18-Pad2) -> Net-(D17H1-Pad2)
- R19 pad 2: unconnected-(R19-Pad2) -> Net-(D18E1-Pad2)
- R2 pad 2: unconnected-(R2-Pad2) -> Net-(D01B1-Pad2)
- R20 pad 2: unconnected-(R20-Pad2) -> Net-(D19H1-Pad2)
- R21 pad 2: unconnected-(R21-Pad2) -> Net-(D20H1-Pad2)
- R22 pad 2: unconnected-(R22-Pad2) -> Net-(R22-Pad2)
- R23 pad 2: unconnected-(R23-Pad2) -> Net-(D22F1-Pad2)
- R24 pad 2: unconnected-(R24-Pad2) -> Net-(R24-Pad2)
- R25 pad 2: unconnected-(R25-Pad2) -> Net-(R25-Pad2)
- R26 pad 2: unconnected-(R26-Pad2) -> Net-(R26-Pad2)
- R27 pad 2: unconnected-(R27-Pad2) -> Net-(D26A1-Pad2)
- R28 pad 2: unconnected-(R28-Pad2) -> Net-(D27A1-Pad2)
- R29 pad 2: unconnected-(R29-Pad2) -> Net-(D28A1-Pad2)
- R3 pad 2: unconnected-(R3-Pad2) -> Net-(D02B1-Pad2)
- R30 pad 2: unconnected-(R30-Pad2) -> Net-(D29B1-Pad2)
- R31 pad 2: unconnected-(R31-Pad2) -> Net-(D30A1-Pad2)
- R32 pad 2: unconnected-(R32-Pad2) -> Net-(D31B1-Pad2)
- R33 pad 2: unconnected-(R33-Pad2) -> Net-(D00F2-Pad2)
- R34 pad 2: unconnected-(R34-Pad2) -> Net-(D01E2-Pad2)
- R35 pad 2: unconnected-(R35-Pad2) -> Net-(D02G2-Pad2)
- R36 pad 2: unconnected-(R36-Pad2) -> Net-(D03G2-Pad2)
- R37 pad 2: unconnected-(R37-Pad2) -> Net-(R37-Pad2)
- R38 pad 2: unconnected-(R38-Pad2) -> Net-(R38-Pad2)
- R39 pad 2: unconnected-(R39-Pad2) -> Net-(R39-Pad2)
- R4 pad 2: unconnected-(R4-Pad2) -> Net-(D03A1-Pad2)
- R40 pad 2: unconnected-(R40-Pad2) -> Net-(R40-Pad2)
- R41 pad 2: unconnected-(R41-Pad2) -> Net-(D08H2-Pad2)
- R42 pad 2: unconnected-(R42-Pad2) -> Net-(D09C2-Pad2)
- R43 pad 2: unconnected-(R43-Pad2) -> Net-(D10C2-Pad2)
- R44 pad 2: unconnected-(R44-Pad2) -> Net-(D11C2-Pad2)
- R45 pad 2: unconnected-(R45-Pad2) -> Net-(D12G2-Pad2)
- R46 pad 2: unconnected-(R46-Pad2) -> Net-(R46-Pad2)
- R47 pad 2: unconnected-(R47-Pad2) -> Net-(D14F2-Pad2)
- R48 pad 2: unconnected-(R48-Pad2) -> Net-(D15F2-Pad2)
- R49 pad 2: unconnected-(R49-Pad2) -> Net-(D16H2-Pad2)
- R5 pad 2: unconnected-(R5-Pad2) -> Net-(D04E1-Pad2)
- R50 pad 2: unconnected-(R50-Pad2) -> Net-(R50-Pad2)
- R51 pad 2: unconnected-(R51-Pad2) -> Net-(D18H2-Pad2)
- R52 pad 2: unconnected-(R52-Pad2) -> Net-(D19H2-Pad2)
- R53 pad 2: unconnected-(R53-Pad2) -> Net-(D20A2-Pad2)
- R54 pad 2: unconnected-(R54-Pad2) -> Net-(D21B2-Pad2)
- R55 pad 2: unconnected-(R55-Pad2) -> Net-(D22G2-Pad2)
- R56 pad 2: unconnected-(R56-Pad2) -> Net-(D23A2-Pad2)
- R57 pad 2: unconnected-(R57-Pad2) -> Net-(R57-Pad2)
- R58 pad 2: unconnected-(R58-Pad2) -> Net-(D25H2-Pad2)
- R59 pad 2: unconnected-(R59-Pad2) -> Net-(R59-Pad2)
- R6 pad 2: unconnected-(R6-Pad2) -> Net-(D05E1-Pad2)
- R60 pad 2: unconnected-(R60-Pad2) -> Net-(D27H2-Pad2)
- R61 pad 2: unconnected-(R61-Pad2) -> Net-(D28H2-Pad2)
- R62 pad 2: unconnected-(R62-Pad2) -> Net-(D29H2-Pad2)
- R63 pad 2: unconnected-(R63-Pad2) -> Net-(R63-Pad2)
- R64 pad 2: unconnected-(R64-Pad2) -> Net-(R64-Pad2)
- R7 pad 2: unconnected-(R7-Pad2) -> Net-(D06H1-Pad2)
- R8 pad 2: unconnected-(R8-Pad2) -> Net-(D07H1-Pad2)
- R9 pad 2: unconnected-(R9-Pad2) -> Net-(D08F1-Pad2)
Routing:
- net Net-(D08F1-Pad2): track 0.00 -> 147.5 mm
- net unconnected-(D31G1-Pad2): track 117.2 -> 0.00 mm
- net Net-(D31B1-Pad2): track 0.00 -> 117.2 mm
- net unconnected-(R64-Pad2): track 116.3 -> 0.00 mm
- net Net-(R64-Pad2): track 0.00 -> 116.3 mm
- net unconnected-(D10D1-Pad2): track 116.3 -> 0.00 mm
- net Net-(D10G1-Pad2): track 0.00 -> 116.3 mm
- net unconnected-(D27B1-Pad2): track 116.1 -> 0.00 mm
- net Net-(D27A1-Pad2): track 0.00 -> 116.1 mm
- net unconnected-(D08G1-Pad2): track 116.0 -> 0.00 mm
- net unconnected-(D29A1-Pad2): track 116.0 -> 0.00 mm
- net Net-(D29B1-Pad2): track 0.00 -> 116.0 mm
- net unconnected-(D00D2-Pad2): track 116.0 -> 0.00 mm
- net Net-(D00F2-Pad2): track 0.00 -> 116.0 mm
- net unconnected-(D01C1-Pad2): track 115.8 -> 0.00 mm
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
Commit message: added more docs
Parts:
- moved C2 245.7 mm to (-51.8, 225.3)
- moved C1 67.2 mm to (-54.6, -2.29), turned to 180 degrees
- moved C11 63.8 mm to (-55.6, 6.86), turned to 90 degrees
- moved C12 60.8 mm to (-55.6, 6.86), turned to 90 degrees
Other:
- board text added: "LED pitch is 0.625{dblquote} = .625 * 25.4 = 15.875mm Board dimension is 571.125 w x 254 h Borders of 10mm on top and 5.875mm on bottom so boards can mate top to bottom preserving LED pitch Height must be exact multiple of LED pitch so boards mate LED grid starts 10mm from top of board All mounting holes are M3.0"
- board text added: "RPi corner radius = 3mm 4 RPi holes are M2.5"
- board text removed: "Board Corner Radius = 3mm All holes are M2.5"
- board text removed: "Board dimensions are on Cmts (Comments) layer. Deselect it in Layers Manager to make them invisible. GPIO connector nets are not connected, these will get updated as per your schematic/netlist."
- board text removed: "LED pitch is 0.625" = .625 * 25.4 = 15.875mm Board dimensions (height) is 16 * led pitch = 264mm top = -10mm bottom = 254 left = right = holes for vertical struts are centered 9 mm to left and right of array so at y = -9mm and (32*pitch) + 9 = 517mm horizontal strut is midpoint of the array, or 8.5 * pitch or 134.94 mm Borders of 10mm on top and 5.875mm on bottom so boards can mate top to bottom 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"
